File: cpu-68008/ide-8bit.brd (EAGLE design)
At the start: 99.7 x 99.7 mm, 15 parts, among them IC101 GAL22V10D, IC201 74HCT245N

Commit message: minor revisions on mouser parts
Parts:
- added C1: 10µF, rcl:SMC_B
- added C2, C3, C4: 100nF, rcl:C0805
- added IC1: ATmega328P, SparkFun-IC-Microcontroller:DIP28
- added SV1: (no value), con-harting-ml:ML6
Connections:
- new net !AVR_RESET: IC1.1, SV1.2
- new net AVR_MISO: SV1.6
- new net AVR_MOSI: SV1.3
- new net AVR_SCK: SV1.4
- net +5V: now also C1.+, C2.1, C3.1, C4.1, IC1.20, IC1.21, IC1.7, SV1.5
- net GND: now also C1.-, C2.2, C3.2, C4.2, IC1.22, IC1.8, SV1.1
Changed lines of the file:
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@@
 <element name="SV101" library="con-lstb" library_urn="urn:adsk.eagle:library:162" package="MA20-2W" package3d_urn="urn:adsk.eagle:package:8363/1" value="" x="62.865" y="5.715" smashed="yes" rot="R180">
 <attribute name="MF" value="" x="23.495" y="48.895" size="1.778" layer="27" rot="R180" display="off"/>
+<attribute name="MOUSER" value="517-30340-5002" x="62.865" y="5.715" size="1.778" layer="27" rot="R180" display="off"/>
 <attribute name="MPN" value="" x="23.495" y="48.895" size="1.778" layer="27" rot="R180" display="off"/>
 <attribute name="NAME" x="88.265" y="9.525" size="1.27" layer="25" ratio="10" rot="R180"/>
@@
 <attribute name="NAME" x="32.385" y="43.18" size="1.27" layer="25"/>
 <attribute name="SPICEPREFIX" value="C" x="33.655" y="41.91" size="1.778" layer="27" display="off"/>
+</element>
+<element name="IC1" library="SparkFun-IC-Microcontroller" package="DIP28" value="ATmega328P" x="-14.605" y="76.2" smashed="yes" rot="R90">
+<attribute name="MOUSER" value="556-ATMEGA328-PU" x="-14.605" y="76.2" size="1.778" layer="27" rot="R90" display="off"/>
+<attribute name="NAME" x="-14.605" y="57.785" size="1.27" layer="25" font="vector" rot="R180" align="bottom-center"/>
+<attribute name="PROD_ID" value="IC-09136" x="-14.605" y="76.2" size="1.778" layer="27" rot="R90" display="off"/>
+</element>
+<element name="SV1" library="con-harting-ml" library_urn="urn:adsk.eagle:library:149" package="ML6" package3d_urn="urn:adsk.eagle:package:6988/1" value="" x="-11.43" y="47.625" smashed="yes">
+<attribute name="MF" value="" x="-11.43" y="47.625" size="1.778" layer="27" display="off"/>
+<attribute name="MPN" value="" x="-11.43" y="47.625" size="1.778" layer="27" display="off"/>
+<attribute name="NAME" x="-19.05" y="52.705" size="1.27" layer="25"/>
+<attribute name="OC_FARNELL" value="unknown" x="-11.43" y="47.625" size="1.778" layer="27" display="off"/>
+<attribute name="OC_NEWARK" value="unknown" x="-11.43" y="47.625" size="1.778" layer="27" display="off"/>
+<attribute name="VALUE" x="-10.795" y="52.705" size="1.778" layer="27" ratio="10"/>
+</element>
+<element name="C1" library="rcl" library_urn="urn:adsk.eagle:library:334" package="SMC_B" package3d_urn="urn:adsk.eagle:package:25920/5" value="10µF" x="-24.765" y="76.2" smashed="yes">
+<attribute name="MOUSER" value="581-TAJB106K020RNJV" x="-31.75" y="83.185" size="1.778" layer="27" display="off"/>
+<attribute name="NAME" x="-26.67" y="78.105" size="1.27" layer="25"/>
+<attribute name="POPULARITY" value="25" x="-31.75" y="83.185" size="1.778" layer="27" display="off"/>
+<attribute name="SPICEPREFIX" value="C" x="-31.75" y="83.185" size="1.778" layer="27" display="off"/>
+</element>
+<element name="C2" library="rcl" library_urn="urn:adsk.eagle:library:334" package="C0805" package3d_urn="urn:adsk.eagle:package:23617/2" value="100nF" x="-24.765" y="71.12" smashed="yes">
+<attribute name="MOUSER" value="710-885012207072" x="-31.115" y="77.47" size="1.778" layer="27" display="off"/>
+<attribute name="NAME" x="-26.035" y="72.39" size="1.27" layer="25"/>
+<attribute name="SPICEPREFIX" value="C" x="-31.115" y="77.47" size="1.778" layer="27" display="off"/>
+</element>
+<element name="C3" library="rcl" library_urn="urn:adsk.eagle:library:334" package="C0805" package3d_urn="urn:adsk.eagle:package:23617/2" value="100nF" x="-13.335" y="37.465" smashed="yes">
+<attribute name="MOUSER" value="710-885012207072" x="-13.335" y="37.465" size="1.778" layer="27" display="off"/>
+<attribute name="NAME" x="-14.605" y="38.735" size="1.27" layer="25"/>
+<attribute name="SPICEPREFIX" value="C" x="-13.335" y="37.465" size="1.778" layer="27" display="off"/>
+</element>
+<element name="C4" library="rcl" library_urn="urn:adsk.eagle:library:334" package="C0805" package3d_urn="urn:adsk.eagle:package:23617/2" value="100nF" x="-24.765" y="66.675" smashed="yes">
+<attribute name="MOUSER" value="710-885012207072" x="-24.765" y="66.675" size="1.778" layer="27" display="off"/>
+<attribute name="NAME" x="-26.035" y="67.945" size="1.27" layer="25"/>
+<attribute name="SPICEPREFIX" value="C" x="-24.765" y="66.675" size="1.778" layer="27" display="off"/>
 </element>
 </elements>
@@
 <wire x1="32.705" y1="38.415" x2="35.56" y2="35.56" width="0.2032" layer="1"/>
 <wire x1="18.2" y1="53.34" x2="5.08" y2="53.34" width="0.2032" layer="1"/>
+<contactref element="IC1" pad="20"/>
+<contactref element="IC1" pad="7"/>
+<contactref element="SV1" pad="5"/>
+<contactref element="C2" pad="1"/>
+<contactref element="C1" pad="+"/>
+<contactref element="C3" pad="1"/>
+<contactref element="IC1" pad="21"/>
+<contactref element="C4" pad="1"/>
+<wire x1="-18.415" y1="77.47" x2="-10.795" y2="74.93" width="0" layer="19" extent="1-1"/>
+<wire x1="-18.415" y1="80.01" x2="-18.415" y2="77.47" width="0" layer="19" extent="1-1"/>
+<wire x1="-25.715" y1="71.12" x2="-18.415" y2="77.47" width="0" layer="19" extent="1-1"/>
+<wire x1="-26.265" y1="76.2" x2="-25.715" y2="71.12" width="0" layer="19" extent="1-1"/>
+<wire x1="5.08" y1="76.835" x2="-10.795" y2="74.93" width="0" layer="19" extent="1-1"/>
+<wire x1="-8.89" y1="46.355" x2="5.08" y2="53.34" width="0" layer="19" extent="1-1"/>
+<wire x1="-14.285" y1="37.465" x2="-8.89" y2="46.355" width="0" layer="19" extent="1-1"/>
+<wire x1="-25.715" y1="66.675" x2="5.08" y2="9.525" width="0" layer="19" extent="1-1"/>
 </signal>
 <signal name="SLOT_D3">
@@
 <contactref element="IC201" pad="10"/>
 <contactref element="C203" pad="2"/>
+<contactref element="IC1" pad="22"/>
+<contactref element="IC1" pad="8"/>
+<contactref element="SV1" pad="1"/>
+<contactref element="C2" pad="2"/>
+<contactref element="C1" pad="-"/>
+<contactref element="C3" pad="2"/>
+<contactref element="C4" pad="2"/>
+<wire x1="-18.415" y1="74.93" x2="-10.795" y2="77.47" width="0" layer="19" extent="1-1"/>
+<wire x1="-23.815" y1="71.12" x2="-18.415" y2="74.93" width="0" layer="19" extent="1-1"/>
+<wire x1="-23.265" y1="76.2" x2="-23.815" y2="71.12" width="0" layer="19" extent="1-1"/>
+<wire x1="0.635" y1="76.835" x2="-10.795" y2="77.47" width="0" layer="19" extent="1-1"/>
+<wire x1="-12.385" y1="37.465" x2="0.635" y2="38.735" width="0" layer="19" extent="1-1"/>
+<wire x1="-13.97" y1="46.355" x2="-12.385" y2="37.465" width="0" layer="19" extent="1-1"/>
+<wire x1="-23.815" y1="66.675" x2="0.635" y2="0.635" width="0" layer="19" extent="1-1"/>
 </signal>
 <signal name="ATA_DIR">
@@
 <wire x1="55.245" y1="27.94" x2="64.135" y2="27.94" width="0.2032" layer="16"/>
 </signal>
+<signal name="!AVR_RESET">
+<contactref element="SV1" pad="2"/>
+<contactref element="IC1" pad="1"/>
+<wire x1="-13.97" y1="48.895" x2="-10.795" y2="59.69" width="0" layer="19" extent="1-1"/>
+</signal>
+<signal name="AVR_SCK">
+<contactref element="SV1" pad="4"/>
+</signal>
+<signal name="AVR_MISO">
+<contactref element="SV1" pad="6"/>
+</signal>
+<signal name="AVR_MOSI">
+<contactref element="SV1" pad="3"/>
+</signal>
 </signals>
