File: cpu-68000/io.brd (EAGLE design)
At the start: 160 x 100 mm, 53 parts, among them IC101 74HC245DW, IC102 74HC85D, IC103 74HC245DW, IC104 74HC245DW, IC105 74HC138D, IC106 GAL22V10D, IC107 74HC243D, IC201 SST39SF010, IC301 XR68C681, IC501 SCC2691, IC502 ATmega328P

Commit message: IO board: 	- Added 82C55 PIO
RAM board:
	- Tweaked tolerances between some traces
	- Fixed naming of parts
Parts:
- removed C116, C3: 100nF, rcl:C0805
- removed QG101: 3.6864 MHz, crystal:DIL08S
- added C103, C303: 10µF, rcl:SMC_B
- added C301, C302: 100nF, rcl:C0805
- added F501, F502: 100mA, 68komputer:WE-MI_1206
- added IC302: 82C55, 68komputer:PLCC-S44
- added QG301: 3.6864 MHz, crystal:DIL08S
- added SV301: (no value), con-lstb:MA07-2W
- added SV401: (no value), con-harting-ml:ML40L
- C102: value 1µF -> 100nF
- C104: value 120µF -> 100nF; device rcl:E2,5-7 -> rcl:C0805
- C105, C2: value 10µF -> 100nF; device rcl:SMC_B -> rcl:C0805
- C106: value 100nF -> 10µF; device rcl:C0805 -> rcl:SMC_B
- C108: value 10µF -> 1µF; device rcl:SMC_B -> rcl:C0805
- C109: value 100nF -> 120µF; device rcl:C0805 -> rcl:E2,5-7
- IC105: value 74HC138D -> 74HC243D; device 74xx-eu:SO16 -> 74xx-eu:SO14
- IC106: value GAL22V10D -> 74HC138D; device 68komputer:DIL24S -> 74xx-eu:SO16
- IC107: value 74HC243D -> GAL22V10D; device 74xx-eu:SO14 -> 68komputer:DIL24S
- IC501: value SCC2691 -> ATmega328P; device 68komputer:DIL24S -> SparkFun-IC-Microcontroller:DIP28
- IC502: value ATmega328P -> SCC2691; device SparkFun-IC-Microcontroller:DIP28 -> 68komputer:DIL24S
- R101: value 10k -> 3k
- R103: value 3k -> 10k
- moved IC106 111.2 mm to (13.5, 60.5)
- moved IC107 110.5 mm to (123.0, 80.0)
- moved R101 98.9 mm to (3.50, 73.0), turned to 90 degrees
- moved C2 91.3 mm to (-41.0, -15.0)
- moved C1 83.2 mm to (-41.0, -8.50)
- moved R103 82.5 mm to (85.5, 82.5), turned to 180 degrees
- moved C102 74.3 mm to (85.5, 80.0), flipped to the top, turned to 180 degrees
- moved C107 71.9 mm to (15.0, 94.0), flipped to the bottom, turned to 90 degrees
- moved C101 69.1 mm to (80.5, 72.0), flipped to the top, turned to 0 degrees
- moved C106 58.7 mm to (22.0, 77.0), turned to 90 degrees
- moved IC501 58.0 mm to (165.5, 25.0), turned to 270 degrees
- moved IC502 58.0 mm to (167.5, 83.0), turned to 90 degrees
- moved IC105 55.0 mm to (12.5, 77.0), turned to 180 degrees
- moved IC301 54.6 mm to (31.5, 25.5), turned to 180 degrees
- moved C108 52.8 mm to (12.5, 94.0), flipped to the bottom
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- renumbered C10 to C502, C117 to C112, C4 to C505, C5 to C507, C6 to C506, C7 to C503, C8 to C501, C9 to C504, R303 to R301, S1 to S101, SV1 to SV501
Connections:
- new net !A_CTS: SV301.1, SV301.9
- new net !B_CTS: SV301.10, SV301.2
- net !AS: now also IC107.11; no longer IC106.11
- net !ATA_CS: now also IC106.14; no longer IC105.14
- net !AVR_RESET: now also IC501.1; no longer IC502.1
- net !CS: now also IC105.1, IC106.4, IC107.14; no longer IC105.4, IC106.14, IC107.1
- net !DTACK: now also IC107.16; no longer IC106.16
- net !DUART_CS: now also IC106.15; no longer IC105.15
- net !EXTI_A: now also IC107.17; no longer IC106.17
- net !EXT_ID: now also IC107.6; no longer IC106.6
- net !I2C_CS: now also IC106.9; no longer IC105.9
- net !LCD_CS: now also IC106.11; no longer IC105.11
- net !LDS: now also IC107.10; no longer IC106.10
- net !PIO_CS: now also IC106.12, IC302.7; no longer IC105.12
- net !PS2_CS: now also IC106.13, IC502.14; no longer IC105.13, IC501.14
- net !PS2_IRQ: now also IC502.13; no longer IC501.13
- net !RD: now also IC107.15, IC302.6, IC502.1; no longer IC106.15, IC501.1
- net !RESET: now also IC107.8; no longer IC106.8
- net !ROM_CS: now also IC106.6, IC107.22; no longer IC105.6, IC106.22
- net !STATUS_CS: now also IC106.10; no longer IC105.10
- net +5V: now also C103.+, C104.1, C105.1, C106.+, C108.1, C109.+, C2.1, C301.1, C302.1, C303.+, F501.1, F502.1, IC105.13, IC105.14, IC106.16, IC107.24, IC302.29, IC501.20, IC501.21, IC501.7, IC502.24, QG301.8, R101.1, SV301.7, SV301.8; no longer C104.+, C105.+, C106.1, C108.+, C109.1, C116.1, C2.+, C3.1, IC105.16, IC106.24, IC107.13, IC107.14, IC501.24, IC502.20, IC502.21, IC502.7, QG101.8, R103.1
- net A17: now also IC105.3; no longer IC107.3
- net A18: now also IC105.4; no longer IC107.4
- net A19: now also IC105.5; no longer IC107.5
- net A8: now also IC107.7; no longer IC106.7
- net A9: now also IC107.4; no longer IC106.4
- net ADDR_MATCH: now also IC107.13; no longer IC106.13
- net ADDR_SET0: now also R105.1; no longer R102.1
- net ADDR_SET1: now also R104.1; no longer R101.1
- net ADDR_SET2: now also R103.1; no longer R104.1
- net ADDR_SET3: now also IC107.5, R102.1; no longer IC106.5, R105.1
- net AVR_MISO: now also IC501.18; no longer IC502.18
- net AVR_MOSI: now also IC501.17; no longer IC502.17
- net AVR_SCK: now also IC501.19; no longer IC502.19
- net A_RX: now also SV301.3
- net A_TX: now also SV301.5
- net BOARD_A0: now also IC302.10
- net BOARD_A1: now also IC302.9
- net BOARD_A13: now also IC106.1
- net BOARD_A14: now also IC106.2; no longer IC105.1
- net BOARD_A15: now also IC106.3; no longer IC105.2
- net BOARD_A16: now also IC105.11; no longer IC105.3, IC107.11
- net BOARD_A17: now also IC105.10; no longer IC107.10
- net BOARD_A18: now also IC105.9; no longer IC107.9
- net BOARD_D0: now also IC201.13, IC302.38
- net BOARD_D1: now also IC201.14, IC302.37
- net BOARD_D2: now also IC201.15, IC302.36
- net BOARD_D3: now also IC201.17, IC302.35
- net BOARD_D4: now also IC201.18, IC302.33
- net BOARD_D5: now also IC201.19, IC302.32
- net BOARD_D6: now also IC201.20, IC302.31
- net BOARD_D7: now also IC201.21, IC302.30
- net B_RX: now also SV301.4
- net B_TX: now also SV301.6
- net GND: now also C103.-, C104.2, C105.2, C106.-, C108.2, C109.-, C2.2, C301.2, C302.2, C303.-, IC105.6, IC105.7, IC106.5, IC106.8, IC107.12, IC302.8, IC501.22, IC501.8, IC502.12, QG301.4, R103.2, SV301.11, SV301.12, SV301.13, SV301.14; no longer C104.-, C105.-, C106.2, C108.-, C109.2, C116.2, C2.-, C3.2, IC105.5, IC105.8, IC106.12, IC107.6, IC107.7, IC501.12, IC502.22, IC502.8, QG101.4, R101.2
- net N$18: now also R101.2; no longer R103.2
- net PS2_UART_RX: now also IC501.3, IC502.2; no longer IC501.2, IC502.3
- net PS2_UART_TX: now also IC501.2, IC502.3; no longer IC501.3, IC502.2
- net R/!W!: now also IC107.9, IC302.40, IC502.23; no longer IC106.9, IC501.23
- net RESET: now also IC302.39, IC502.11; no longer IC501.11
- net SLOT_A0: now also IC502.8; no longer IC501.8
- net SLOT_A1: now also IC502.7; no longer IC501.7
- net SLOT_A2: now also IC502.6; no longer IC501.6
- net SLOT_D0: now also IC502.22; no longer IC201.13, IC501.22
- net SLOT_D1: now also IC502.21; no longer IC201.14, IC501.21
- net SLOT_D2: now also IC502.20; no longer IC201.15, IC501.20
- net SLOT_D3: now also IC502.19; no longer IC201.17, IC501.19
- net SLOT_D4: now also IC502.18; no longer IC201.18, IC501.18
- net SLOT_D5: now also IC502.17; no longer IC201.19, IC501.17
- net SLOT_D6: now also IC502.16; no longer IC201.20, IC501.16
- net SLOT_D7: now also IC502.15; no longer IC201.21, IC501.15
- net UART_CLK: now also IC502.9, QG301.5; no longer IC501.9, QG101.5
Routing:
- net BOARD_D3: track 0.00 -> 33.1 mm
- net BOARD_D6: track 0.00 -> 21.3 mm
- net BOARD_D7: track 0.00 -> 20.2 mm
- net BOARD_D4: track 0.00 -> 20.2 mm
- net BOARD_D2: track 0.00 -> 19.4 mm
- net +5V: track 197.7 -> 217.0 mm
- net BOARD_D1: track 0.00 -> 15.7 mm, vias 0 -> 1
- net BOARD_D0: track 0.00 -> 15.6 mm
- net BOARD_D5: track 0.00 -> 15.5 mm
- net UART_CLK: track 0.00 -> 13.6 mm
Other:
- board text added: "68komputer Multi IO Board (from 11, 2.5)"
- board text removed: "68komputer Multi IO Board"
