File: cpu-68000/io.sch (EAGLE design)
At the start: 72 parts, among them IC101 74HC245DW, IC102 74HC245DW, IC103 74HC245DW, IC104 74HC245DW, IC105 74HC138D, IC106 GAL22V10D, IC107 74HC243D

Commit message: CPU board: 	- Clean up some traces
IO board:
	- Started work on super IO board
	- UARTs, parallel port, PS/2 keyboard/mouse interface, I2C

2MB RAM Expansion:
	- Added some address decoding
Parts:
- removed C112, C204, C205, C207, C208, C210, C211, C301, C302, C304, C305, C307, C308, C310, C311: 100nF, rcl:C-EUC0805
- removed C203, C206, C209, C212, C303, C306, C309, C312: 10µF, rcl:CPOL-EUSMCB
- removed IC202, IC203, IC204, IC205, IC206, IC207, IC208, IC302, IC303, IC304, IC305, IC306, IC307, IC308: (no value), 68komputer:CY62128BSOIC32-450
- added C1, C10, C117, C3, C4, C6, C8, C9: 100nF, rcl:C-EUC0805
- added C2, C5, C7: 10µF, rcl:CPOL-EUSMCB
- added IC501: SCC2691, 68komputer:SCC2691
- added IC502: ATmega328P, SparkFun-IC-Microcontroller:ATMEGA328P_PDIP
- added QG101: 3.6864 MHz, crystal:XO-8
- added R104, R105, R303: 10k, rcl:R-EU_R2012
- added SV1: (no value), con-harting-ml:ML6
- C202: value 100nF -> 10µF; device rcl:C-EUC0805 -> rcl:CPOL-EUSMCB; MOUSER 710-885012207072 -> 581-TAJB106K020RNJV
- IC102: value 74HC245DW -> 74HC85D; device 74xx-eu:74HC245DW -> 74xx-eu:74HC85D; MOUSER 595-SN74HC245DWR -> 771-74HC138D
- IC105: MOUSER 595-SN74HC138DG4 -> 771-74HC138D
- IC201: value (none) -> SST39SF010; device 68komputer:CY62128BSOIC32-450 -> 68komputer:SST39SF0X0PLCC32-SOCKET; MOUSER (none) -> 579-SST3910A554INHET; MOUSER_SOCKET (none) -> 437-5408803224008
- IC301: value (none) -> XR68C681; device 68komputer:CY62128BSOIC32-450 -> 68komputer:MC68681PLCC44-SOCKET; MOUSER (none) -> 701-XR68C681CJ-F; MOUSER_SOCKET (none) -> 940-44-044-24-000000
- S1: device switch-dil:DP02 -> switch-dil:DP04; MOUSER (none) -> 653-A6FR-2104
Connections:
- removed net !LOE: IC106.IO20, IC201.!OE, IC202.!OE, IC203.!OE, IC204.!OE, IC205.!OE, IC206.!OE, IC207.!OE, IC208.!OE
- removed net !RAM_CS0: IC105A.Y0, IC201.!CE1, IC301.!CE1
- removed net !RAM_CS1: IC105A.Y1, IC202.!CE1, IC302.!CE1
- removed net !RAM_CS2: IC105A.Y2, IC203.!CE1, IC303.!CE1
- removed net !RAM_CS3: IC105A.Y3, IC204.!CE1, IC304.!CE1
- removed net !RAM_CS4: IC105A.Y4, IC205.!CE1, IC305.!CE1
- removed net !RAM_CS5: IC105A.Y5, IC206.!CE1, IC306.!CE1
- removed net !RAM_CS6: IC105A.Y6, IC207.!CE1, IC307.!CE1
- removed net !RAM_CS7: IC105A.Y7, IC208.!CE1, IC308.!CE1
- removed net !UOE: IC106.IO22, IC301.!OE, IC302.!OE, IC303.!OE, IC304.!OE, IC305.!OE, IC306.!OE, IC307.!OE, IC308.!OE
- removed net !UWE: IC106.IO23, IC301.!WE, IC302.!WE, IC303.!WE, IC304.!WE, IC305.!WE, IC306.!WE, IC307.!WE, IC308.!WE
- removed net N$5: IC106.IO19
- removed net N$6: IC106.IO18
- removed net N$7: IC106.IO17
- removed net RAM_A0: IC103A.B1, IC201.A0, IC202.A0, IC203.A0, IC204.A0, IC205.A0, IC206.A0, IC207.A0, IC208.A0, IC301.A0, IC302.A0, IC303.A0, IC304.A0, IC305.A0, IC306.A0, IC307.A0, IC308.A0
- removed net RAM_A1: IC103A.B2, IC201.A1, IC202.A1, IC203.A1, IC204.A1, IC205.A1, IC206.A1, IC207.A1, IC208.A1, IC301.A1, IC302.A1, IC303.A1, IC304.A1, IC305.A1, IC306.A1, IC307.A1, IC308.A1
- removed net RAM_A10: IC104A.B3, IC201.A10, IC202.A10, IC203.A10, IC204.A10, IC205.A10, IC206.A10, IC207.A10, IC208.A10, IC301.A10, IC302.A10, IC303.A10, IC304.A10, IC305.A10, IC306.A10, IC307.A10, IC308.A10
- removed net RAM_A11: IC104A.B4, IC201.A11, IC202.A11, IC203.A11, IC204.A11, IC205.A11, IC206.A11, IC207.A11, IC208.A11, IC301.A11, IC302.A11, IC303.A11, IC304.A11, IC305.A11, IC306.A11, IC307.A11, IC308.A11
- removed net RAM_A12: IC104A.B5, IC201.A12, IC202.A12, IC203.A12, IC204.A12, IC205.A12, IC206.A12, IC207.A12, IC208.A12, IC301.A12, IC302.A12, IC303.A12, IC304.A12, IC305.A12, IC306.A12, IC307.A12, IC308.A12
- removed net RAM_A13: IC104A.B6, IC201.A13, IC202.A13, IC203.A13, IC204.A13, IC205.A13, IC206.A13, IC207.A13, IC208.A13, IC301.A13, IC302.A13, IC303.A13, IC304.A13, IC305.A13, IC306.A13, IC307.A13, IC308.A13
- removed net RAM_A14: IC104A.B7, IC201.A14, IC202.A14, IC203.A14, IC204.A14, IC205.A14, IC206.A14, IC207.A14, IC208.A14, IC301.A14, IC302.A14, IC303.A14, IC304.A14, IC305.A14, IC306.A14, IC307.A14, IC308.A14
- removed net RAM_A15: IC104A.B8, IC201.A15, IC202.A15, IC203.A15, IC204.A15, IC205.A15, IC206.A15, IC207.A15, IC208.A15, IC301.A15, IC302.A15, IC303.A15, IC304.A15, IC305.A15, IC306.A15, IC307.A15, IC308.A15
- removed net RAM_A16: IC107A.B1, IC201.A16, IC202.A16, IC203.A16, IC204.A16, IC205.A16, IC206.A16, IC207.A16, IC208.A16, IC301.A16, IC302.A16, IC303.A16, IC304.A16, IC305.A16, IC306.A16, IC307.A16, IC308.A16
- removed net RAM_A2: IC103A.B3, IC201.A2, IC202.A2, IC203.A2, IC204.A2, IC205.A2, IC206.A2, IC207.A2, IC208.A2, IC301.A2, IC302.A2, IC303.A2, IC304.A2, IC305.A2, IC306.A2, IC307.A2, IC308.A2
- removed net RAM_A3: IC103A.B4, IC201.A3, IC202.A3, IC203.A3, IC204.A3, IC205.A3, IC206.A3, IC207.A3, IC208.A3, IC301.A3, IC302.A3, IC303.A3, IC304.A3, IC305.A3, IC306.A3, IC307.A3, IC308.A3
- removed net RAM_A4: IC103A.B5, IC201.A4, IC202.A4, IC203.A4, IC204.A4, IC205.A4, IC206.A4, IC207.A4, IC208.A4, IC301.A4, IC302.A4, IC303.A4, IC304.A4, IC305.A4, IC306.A4, IC307.A4, IC308.A4
- removed net RAM_A5: IC103A.B6, IC201.A5, IC202.A5, IC203.A5, IC204.A5, IC205.A5, IC206.A5, IC207.A5, IC208.A5, IC301.A5, IC302.A5, IC303.A5, IC304.A5, IC305.A5, IC306.A5, IC307.A5, IC308.A5
- removed net RAM_A6: IC103A.B7, IC201.A6, IC202.A6, IC203.A6, IC204.A6, IC205.A6, IC206.A6, IC207.A6, IC208.A6, IC301.A6, IC302.A6, IC303.A6, IC304.A6, IC305.A6, IC306.A6, IC307.A6, IC308.A6
- removed net RAM_A7: IC103A.B8, IC201.A7, IC202.A7, IC203.A7, IC204.A7, IC205.A7, IC206.A7, IC207.A7, IC208.A7, IC301.A7, IC302.A7, IC303.A7, IC304.A7, IC305.A7, IC306.A7, IC307.A7, IC308.A7
- removed net RAM_A8: IC104A.B1, IC201.A8, IC202.A8, IC203.A8, IC204.A8, IC205.A8, IC206.A8, IC207.A8, IC208.A8, IC301.A8, IC302.A8, IC303.A8, IC304.A8, IC305.A8, IC306.A8, IC307.A8, IC308.A8
- removed net RAM_A9: IC104A.B2, IC201.A9, IC202.A9, IC203.A9, IC204.A9, IC205.A9, IC206.A9, IC207.A9, IC208.A9, IC301.A9, IC302.A9, IC303.A9, IC304.A9, IC305.A9, IC306.A9, IC307.A9, IC308.A9
- removed net RAM_D0: IC101A.B1, IC201.D0, IC202.D0, IC203.D0, IC204.D0, IC205.D0, IC206.D0, IC207.D0, IC208.D0
- removed net RAM_D1: IC101A.B2, IC201.D1, IC202.D1, IC203.D1, IC204.D1, IC205.D1, IC206.D1, IC207.D1, IC208.D1
- removed net RAM_D10: IC102A.B3, IC301.D2, IC302.D2, IC303.D2, IC304.D2, IC305.D2, IC306.D2, IC307.D2, IC308.D2
- removed net RAM_D11: IC102A.B4, IC301.D3, IC302.D3, IC303.D3, IC304.D3, IC305.D3, IC306.D3, IC307.D3, IC308.D3
- removed net RAM_D12: IC102A.B5, IC301.D4, IC302.D4, IC303.D4, IC304.D4, IC305.D4, IC306.D4, IC307.D4, IC308.D4
- removed net RAM_D13: IC102A.B6, IC301.D5, IC302.D5, IC303.D5, IC304.D5, IC305.D5, IC306.D5, IC307.D5, IC308.D5
- removed net RAM_D14: IC102A.B7, IC301.D6, IC302.D6, IC303.D6, IC304.D6, IC305.D6, IC306.D6, IC307.D6, IC308.D6
- removed net RAM_D15: IC102A.B8, IC301.D7, IC302.D7, IC303.D7, IC304.D7, IC305.D7, IC306.D7, IC307.D7, IC308.D7
- removed net RAM_D2: IC101A.B3, IC201.D2, IC202.D2, IC203.D2, IC204.D2, IC205.D2, IC206.D2, IC207.D2, IC208.D2
- removed net RAM_D3: IC101A.B4, IC201.D3, IC202.D3, IC203.D3, IC204.D3, IC205.D3, IC206.D3, IC207.D3, IC208.D3
- removed net RAM_D4: IC101A.B5, IC201.D4, IC202.D4, IC203.D4, IC204.D4, IC205.D4, IC206.D4, IC207.D4, IC208.D4
- removed net RAM_D5: IC101A.B6, IC201.D5, IC202.D5, IC203.D5, IC204.D5, IC205.D5, IC206.D5, IC207.D5, IC208.D5
- removed net RAM_D6: IC101A.B7, IC201.D6, IC202.D6, IC203.D6, IC204.D6, IC205.D6, IC206.D6, IC207.D6, IC208.D6
- removed net RAM_D7: IC101A.B8, IC201.D7, IC202.D7, IC203.D7, IC204.D7, IC205.D7, IC206.D7, IC207.D7, IC208.D7
- removed net RAM_D8: IC102A.B1, IC301.D0, IC302.D0, IC303.D0, IC304.D0, IC305.D0, IC306.D0, IC307.D0, IC308.D0
- removed net RAM_D9: IC102A.B2, IC301.D1, IC302.D1, IC303.D1, IC304.D1, IC305.D1, IC306.D1, IC307.D1, IC308.D1
- new net !68681_IRQ: IC301.!INTR, R303.1
- new net !ATA_CS: IC105A.Y1
- new net !AVR_RESET: IC502.PC6(/RESET), SV1.2
- new net !DUART_CS: IC105A.Y0, IC301.!CS
- new net !I2C_CS: IC105A.Y6
- new net !LCD_CS: IC105A.Y4
- new net !PIO_CS: IC105A.Y3
- new net !PS2_CS: IC105A.Y2, IC501.!CS
- new net !PS2_IRQ: IC501.!IRQ
- new net !ROM_CS: IC105A.G1, IC106.IO22, IC201.!CS
- new net !STATUS_CS: IC105A.Y5
- new net ADDR_MATCH: IC102A.A=B_O, IC106.IN13
- new net ADDR_SET2: IC102A.B2, R104.1, S1.6
- new net ADDR_SET3: IC106.IN5, R105.1, S1.5
- new net AVR_MISO: IC502.PB4(MISO), SV1.6
- new net AVR_MOSI: IC502.PB3(MOSI/OC2), SV1.3
- new net AVR_SCK: IC502.PB5(SCK), SV1.4
- new net A_RX: IC301.RXDA
- new net A_TX: IC301.TXDA
- new net BOARD_A0: IC103A.B1, IC201.A0, IC301.A1
- new net BOARD_A1: IC103A.B2, IC201.A1, IC301.A2
- new net BOARD_A10: IC104A.B3, IC201.A10
- new net BOARD_A11: IC104A.B4, IC201.A11
- new net BOARD_A12: IC104A.B5, IC201.A12
- new net BOARD_A13: IC104A.B6, IC201.A13
- new net BOARD_A14: IC104A.B7, IC105A.A, IC201.A14
- new net BOARD_A15: IC104A.B8, IC105A.B, IC201.A15
- new net BOARD_A16: IC105A.C, IC107A.B1
- new net BOARD_A17: IC107A.B2
- new net BOARD_A18: IC107A.B3
- new net BOARD_A2: IC103A.B3, IC201.A2, IC301.A3
- new net BOARD_A3: IC103A.B4, IC201.A3, IC301.A4
- new net BOARD_A4: IC103A.B5, IC201.A4
- new net BOARD_A5: IC103A.B6, IC201.A5
- new net BOARD_A6: IC103A.B7, IC201.A6
- new net BOARD_A7: IC103A.B8, IC201.A7
- new net BOARD_A8: IC104A.B1, IC201.A8
- new net BOARD_A9: IC104A.B2, IC201.A9
- new net BOARD_D0: IC101A.B1, IC301.D0
- new net BOARD_D1: IC101A.B2, IC301.D1
- new net BOARD_D2: IC101A.B3, IC301.D2
- new net BOARD_D3: IC101A.B4, IC301.D3
- new net BOARD_D4: IC101A.B5, IC301.D4
- new net BOARD_D5: IC101A.B6, IC301.D5
- new net BOARD_D6: IC101A.B7, IC301.D6
- new net BOARD_D7: IC101A.B8, IC301.D7
- new net B_RX: IC301.RXDB
- new net B_TX: IC301.TXDB
- new net PS2_UART_RX: IC501.RXD, IC502.PD1(TXD)
- new net PS2_UART_TX: IC501.TXD, IC502.PD0(RXD)
- new net RESET: IC501.RESET
- new net SLOT_A0: IC501.A0
- new net SLOT_A1: IC501.A1
- new net SLOT_A2: IC501.A2
- new net SLOT_D0: IC201.DQ0, IC501.D0
- new net SLOT_D1: IC201.DQ1, IC501.D1
- new net SLOT_D2: IC201.DQ2, IC501.D2
- new net SLOT_D3: IC201.DQ3, IC501.D3
- new net SLOT_D4: IC201.DQ4, IC501.D4
- new net SLOT_D5: IC201.DQ5, IC501.D5
- new net SLOT_D6: IC201.DQ6, IC501.D6
- new net SLOT_D7: IC201.DQ7, IC501.D7
- new net UART_CLK: IC301.X1/CLK, IC501.X1/CLK, QG101.OUT
- net !AS: now also IC106.IN11; no longer IC106.IN5
- net !CS: no longer IC102A.G
- net !DTACK: now also IC301.!DTACK
- net !EXTI_A: now also IC106.IO17
- net !EXT_ID: now also IC106.IN6
- net !LDS: now also IC106.IN10; no longer IC106.IN3
- net !LWE: now also IC301.R/!W; no longer IC106.IO21, IC201.!WE, IC202.!WE, IC203.!WE, IC204.!WE, IC205.!WE, IC206.!WE, IC207.!WE, IC208.!WE
- net !RD: now also IC201.!OE, IC501.!RD; no longer IC102A.DIR
- net !RESET: now also IC106.IN8, IC301.!RESET; no longer IC106.IN1/CLK
- net !UDS: no longer IC106.IN4
- net +5V: now also C1.1, C10.1, C117.1, C2.+, C202.+, C3.1, C4.1, C5.+, C6.1, C7.+, C8.1, C9.1, IC102A.A=B_I, IC102A.B3, IC301.!IACK, IC501.VCC, IC502.AREF, IC502.AVCC, IC502.VCC, QG101.VCC, R303.2, S1.3, S1.4, SV1.5; no longer C112.1, C202.1, C203.+, C204.1, C205.1, C206.+, C207.1, C208.1, C209.+, C210.1, C211.1, C212.+, C301.1, C302.1, C303.+, C304.1, C305.1, C306.+, C307.1, C308.1, C309.+, C310.1, C311.1, C312.+, IC105A.G1, IC201.CE2, IC202.CE2, IC202.VCC, IC203.CE2, IC203.VCC, IC204.CE2, IC204.VCC, IC205.CE2, IC205.VCC, IC206.CE2, IC206.VCC, IC207.CE2, IC207.VCC, IC208.CE2, IC208.VCC, IC301.CE2, IC302.CE2, IC302.VCC, IC303.CE2, IC303.VCC, IC304.CE2, IC304.VCC, IC305.CE2, IC305.VCC, IC306.CE2, IC306.VCC, IC307.CE2, IC307.VCC, IC308.CE2, IC308.VCC
- net A18: now also IC107A.A2; no longer IC105A.A
- net A19: now also IC107A.A3; no longer IC105A.B, IC106.IN6
- net A20: now also IC102A.A0; no longer IC105A.C, IC106.IN7
- net A21: now also IC102A.A1; no longer IC106.IN8
- net A22: now also IC102A.A2; no longer IC106.IN9
- net A23: now also IC102A.A3; no longer IC106.IN13
- net A8: now also IC106.IN7
- net A9: now also IC106.IN4
- net ADDR_SET0: now also IC102A.B0, S1.8; no longer IC106.IN10, S1.4
- net ADDR_SET1: now also IC102A.B1, S1.7; no longer IC106.IN11, S1.3
- net D10: no longer IC102A.A3
- net D11: no longer IC102A.A4
- net D12: no longer IC102A.A5
- net D13: no longer IC102A.A6
- net D14: no longer IC102A.A7
- net D15: no longer IC102A.A8
- net D8: no longer IC102A.A1
- net D9: no longer IC102A.A2
- net GND: now also C1.2, C10.2, C117.2, C2.-, C202.-, C3.2, C4.2, C5.-, C6.2, C7.-, C8.2, C9.2, IC102A.A<B_I, IC102A.A>B_I, IC201.A16, IC201.A17, IC201.A18, IC501.GND, IC502.GND, QG101.GND, R104.2, R105.2, SV1.1; no longer C112.2, C202.2, C203.-, C204.2, C205.2, C206.-, C207.2, C208.2, C209.-, C210.2, C211.2, C212.-, C301.2, C302.2, C303.-, C304.2, C305.2, C306.-, C307.2, C308.2, C309.-, C310.2, C311.2, C312.-, IC107A.A2, IC107A.A3, IC202.GND, IC203.GND, IC204.GND, IC205.GND, IC206.GND, IC207.GND, IC208.GND, IC302.GND, IC303.GND, IC304.GND, IC305.GND, IC306.GND, IC307.GND, IC308.GND
- net R/!W!: now also IC106.IN9, IC201.!WE, IC501.!WR; no longer IC106.IN2

Commit message: IO board: 	- Added 82C55 PIO
RAM board:
	- Tweaked tolerances between some traces
	- Fixed naming of parts
Parts:
- removed C116: 100nF, rcl:C-EUC0805
- added C103, C303: 10µF, rcl:CPOL-EUSMCB
- added C301: 100nF, rcl:C-EUC0805
- added F501, F502: 100mA, 68komputer:FUSE1206
- added IC302: 82C55, 68komputer:82C55PLCC44-SOCKET
- added SV301: (no value), con-lstb:MA07-2W
- added SV401: (no value), con-harting-ml:ML40L
- C102: value 1µF -> 100nF; MOUSER 710-885012207078 -> 710-885012207072
- C104: value 120µF -> 100nF; device rcl:CPOL-EUE2.5-7 -> rcl:C-EUC0805; MOUSER 710-860020373007 -> 710-885012207072
- C105, C2: value 10µF -> 100nF; device rcl:CPOL-EUSMCB -> rcl:C-EUC0805; MOUSER 581-TAJB106K020RNJV -> 710-885012207072
- C106: value 100nF -> 10µF; device rcl:C-EUC0805 -> rcl:CPOL-EUSMCB; MOUSER 710-885012207072 -> 581-TAJB106K020RNJV
- C108: value 10µF -> 1µF; device rcl:CPOL-EUSMCB -> rcl:C-EUC0805; MOUSER 581-TAJB106K020RNJV -> 710-885012207078
- C109: value 100nF -> 120µF; device rcl:C-EUC0805 -> rcl:CPOL-EUE2.5-7; MOUSER 710-885012207072 -> 710-860020373007
- IC105: value 74HC138D -> 74HC243D; device 74xx-eu:74HC138D -> 74xx-eu:74HC243D; MOUSER 771-74HC138D -> 595-CD74HC243M96
- IC106: value GAL22V10D -> 74HC138D; device 68komputer:GAL22V10DIP24 -> 74xx-eu:74HC138D; MOUSER (none) -> 595-SN74HC138DG4; MOUSER_SOCKET 575-1104732441001000 -> (none)
- IC107: value 74HC243D -> GAL22V10D; device 74xx-eu:74HC243D -> 68komputer:GAL22V10DIP24; MOUSER 595-CD74HC243M96 -> (none); MOUSER_SOCKET (none) -> 575-1104732441001000
- IC501: value SCC2691 -> ATmega328P; device 68komputer:SCC2691 -> SparkFun-IC-Microcontroller:ATMEGA328P_PDIP; MOUSER (none) -> 556-ATMEGA328-PU; MOUSER_SOCKET 575-1104732441001000 -> (none)
- IC502: value ATmega328P -> SCC2691; device SparkFun-IC-Microcontroller:ATMEGA328P_PDIP -> 68komputer:SCC2691; MOUSER 556-ATMEGA328-PU -> (none); MOUSER_SOCKET (none) -> 575-1104732441001000
- R101: value 10k -> 3k; MOUSER 652-CR0805FX-1002ELF -> 652-CR0805JW-302ELF
- R103: value 3k -> 10k; MOUSER 652-CR0805JW-302ELF -> 652-CR0805FX-1002ELF
- renumbered C10 to C502, C117 to C112, C3 to C302, C4 to C505, C5 to C507, C6 to C506, C7 to C503, C8 to C501, C9 to C504, QG101 to QG301, R303 to R301, S1 to S101, SV1 to SV501
Connections:
- new net !A_CTS: SV301.1, SV301.9
- new net !B_CTS: SV301.10, SV301.2
- net !AS: now also IC107.IN11; no longer IC106.IN11
- net !ATA_CS: now also IC106A.Y1; no longer IC105A.Y1
- net !AVR_RESET: now also IC501.PC6(/RESET); no longer IC502.PC6(/RESET)
- net !CS: now also IC105A.GAB, IC106A.G2A, IC107.IO14; no longer IC105A.G2A, IC106.IO14, IC107A.GAB
- net !DTACK: now also IC107.IO16; no longer IC106.IO16
- net !DUART_CS: now also IC106A.Y0; no longer IC105A.Y0
- net !EXTI_A: now also IC107.IO17; no longer IC106.IO17
- net !EXT_ID: now also IC107.IN6; no longer IC106.IN6
- net !I2C_CS: now also IC106A.Y6; no longer IC105A.Y6
- net !LCD_CS: now also IC106A.Y4; no longer IC105A.Y4
- net !LDS: now also IC107.IN10; no longer IC106.IN10
- net !PIO_CS: now also IC106A.Y3, IC302.!CS; no longer IC105A.Y3
- net !PS2_CS: now also IC106A.Y2, IC502.!CS; no longer IC105A.Y2, IC501.!CS
- net !PS2_IRQ: now also IC502.!IRQ; no longer IC501.!IRQ
- net !RD: now also IC107.IO15, IC302.!RD, IC502.!RD; no longer IC106.IO15, IC501.!RD
- net !RESET: now also IC107.IN8; no longer IC106.IN8
- net !ROM_CS: now also IC106A.G1, IC107.IO22; no longer IC105A.G1, IC106.IO22
- net !STATUS_CS: now also IC106A.Y5; no longer IC105A.Y5
- net +5V: now also C103.+, C104.1, C105.1, C106.+, C108.1, C109.+, C2.1, C301.1, C303.+, F501.1, F502.1, IC105A.GBA, IC106P.VCC, IC107.VCC, IC302.VCC, IC501.AREF, IC501.AVCC, R101.1, SV301.7, SV301.8; no longer C104.+, C105.+, C106.1, C108.+, C109.1, C116.1, C2.+, IC106.VCC, IC107A.GBA, IC107P.VCC, IC502.AREF, IC502.AVCC, R103.1
- net A17: now also IC105A.A1; no longer IC107A.A1
- net A18: now also IC105A.A2; no longer IC107A.A2
- net A19: now also IC105A.A3; no longer IC107A.A3
- net A8: now also IC107.IN7; no longer IC106.IN7
- net A9: now also IC107.IN4; no longer IC106.IN4
- net ADDR_MATCH: now also IC107.IN13; no longer IC106.IN13
- net ADDR_SET0: now also R105.1; no longer R102.1
- net ADDR_SET1: now also R104.1; no longer R101.1
- net ADDR_SET2: now also R103.1; no longer R104.1
- net ADDR_SET3: now also IC107.IN5, R102.1; no longer IC106.IN5, R105.1
- net AVR_MISO: now also IC501.PB4(MISO); no longer IC502.PB4(MISO)
- net AVR_MOSI: now also IC501.PB3(MOSI/OC2); no longer IC502.PB3(MOSI/OC2)
- net AVR_SCK: now also IC501.PB5(SCK); no longer IC502.PB5(SCK)
- net A_RX: now also SV301.3
- net A_TX: now also SV301.5
- net BOARD_A0: now also IC302.A0
- net BOARD_A1: now also IC302.A1
- net BOARD_A13: now also IC106A.A
- net BOARD_A14: now also IC106A.B; no longer IC105A.A
- net BOARD_A15: now also IC106A.C; no longer IC105A.B
- net BOARD_A16: now also IC105A.B1; no longer IC105A.C, IC107A.B1
- net BOARD_A17: now also IC105A.B2; no longer IC107A.B2
- net BOARD_A18: now also IC105A.B3; no longer IC107A.B3
- net BOARD_D0: now also IC201.DQ0, IC302.D0
- net BOARD_D1: now also IC201.DQ1, IC302.D1
- net BOARD_D2: now also IC201.DQ2, IC302.D2
- net BOARD_D3: now also IC201.DQ3, IC302.D3
- net BOARD_D4: now also IC201.DQ4, IC302.D4
- net BOARD_D5: now also IC201.DQ5, IC302.D5
- net BOARD_D6: now also IC201.DQ6, IC302.D6
- net BOARD_D7: now also IC201.DQ7, IC302.D7
- net B_RX: now also SV301.4
- net B_TX: now also SV301.6
- net GND: now also C103.-, C104.2, C105.2, C106.-, C108.2, C109.-, C2.2, C301.2, C303.-, IC105A.A4, IC106A.G2B, IC106P.GND, IC107.GND, IC302.GND, R103.2, SV301.11, SV301.12, SV301.13, SV301.14; no longer C104.-, C105.-, C106.2, C108.-, C109.2, C116.2, C2.-, IC105A.G2B, IC106.GND, IC107A.A4, IC107P.GND, R101.2
- net N$18: now also R101.2; no longer R103.2
- net PS2_UART_RX: now also IC501.PD1(TXD), IC502.RXD; no longer IC501.RXD, IC502.PD1(TXD)
- net PS2_UART_TX: now also IC501.PD0(RXD), IC502.TXD; no longer IC501.TXD, IC502.PD0(RXD)
- net R/!W!: now also IC107.IN9, IC302.!WR, IC502.!WR; no longer IC106.IN9, IC501.!WR
- net RESET: now also IC302.RESET, IC502.RESET; no longer IC501.RESET
- net SLOT_A0: now also IC502.A0; no longer IC501.A0
- net SLOT_A1: now also IC502.A1; no longer IC501.A1
- net SLOT_A2: now also IC502.A2; no longer IC501.A2
- net SLOT_D0: now also IC502.D0; no longer IC201.DQ0, IC501.D0
- net SLOT_D1: now also IC502.D1; no longer IC201.DQ1, IC501.D1
- net SLOT_D2: now also IC502.D2; no longer IC201.DQ2, IC501.D2
- net SLOT_D3: now also IC502.D3; no longer IC201.DQ3, IC501.D3
- net SLOT_D4: now also IC502.D4; no longer IC201.DQ4, IC501.D4
- net SLOT_D5: now also IC502.D5; no longer IC201.DQ5, IC501.D5
- net SLOT_D6: now also IC502.D6; no longer IC201.DQ6, IC501.D6
- net SLOT_D7: now also IC502.D7; no longer IC201.DQ7, IC501.D7
- net UART_CLK: now also IC502.X1/CLK; no longer IC501.X1/CLK
