File: cpu-68000/cpu-68000.brd (EAGLE design)
At the start: 160 x 100 mm, 105 parts, among them IC201 AS6C4008, IC202 AS6C4008, IC203 39SF040, IC204 39SF040, IC301 XR68C681, IC302 DS1244Y, IC303 MAX232, IC401 GAL22V10, IC402 GAL22V10, IC403 74HC14D, IC404 LM3724, IC405 74HC175D, J201 POWER_JACK, Q301 3.6864 MHz

Commit message: Rev01 of CPU-68000 and 2MB SRAM board sent to production
Parts:
- removed C1: 1µF, rcl:C0805
- added C106: 10µF, rcl:SMC_B
- added LED101, LED102: (no value), led:CHIPLED_1206
- added R121, R122: 10k, rcl:R2012
- added SJ301, SJ302, SJ303, SJ304: (no value), jumper:SJ_2W
- C102: value 100nF -> 1µF
- C104: value 10µF -> 100nF; device rcl:SMC_B -> rcl:C0805
- R101, R102, R308, R309, R310: value 10k -> 3k
- R312, R313, R314: value 3k -> 10k
- moved R106 126.7 mm to (16.5, 71.1)
- moved R105 124.0 mm to (16.5, 62.2), turned to 90 degrees
- moved R102 97.9 mm to (104.0, 77.5), flipped to the top, turned to 270 degrees
- moved R101 91.0 mm to (100.0, 77.5), flipped to the top, turned to 270 degrees
- moved R113 68.5 mm to (141.8, 68.6), turned to 90 degrees
- moved R114 63.5 mm to (139.2, 68.6)
- moved C105 41.1 mm to (40.0, 62.2), turned to 270 degrees
- moved R104 40.0 mm to (17.8, 31.1), turned to 90 degrees
- moved C101 39.9 mm to (14.0, 94.0), turned to 90 degrees
- moved C103 36.2 mm to (4.45, 55.2)
- moved C102 27.8 mm to (11.5, 94.0), turned to 90 degrees
- moved R308 22.9 mm to (115.7, 17.1), flipped to the top
- moved R117 22.0 mm to (89.5, 32.4), turned to 90 degrees
- moved R311 21.7 mm to (93.3, 22.2), turned to 180 degrees
- moved R116 21.0 mm to (87.0, 32.4), turned to 90 degrees
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Connections:
- new net COM0_CTS_PIN: SJ303.2, X301.8
- new net COM0_RTS_PIN: SJ301.2, X301.7
- new net COM0_RX_PIN: SJ302.2, X301.2
- new net COM0_TX_PIN: SJ304.2, X301.3
- new net N$18: LED101.A, R101.1
- new net N$19: LED102.A, R102.1
- net !BR: now also R106.1; no longer R104.1
- net !DTACK: now also R103.1; no longer R101.1
- net !HALT: now also LED102.C, R105.1; no longer R103.1
- net !RESET: now also LED101.C, R104.1; no longer R102.1
- net +5V: now also C104.1, C106.+, R105.2, R106.2; no longer C1.1, C104.+
- net COM0_CTS: now also SJ301.3, SJ303.3; no longer X301.8
- net COM0_RTS: now also SJ301.1, SJ303.1; no longer X301.7
- net COM0_RX: now also SJ302.3, SJ304.3; no longer X301.2
- net COM0_TX: now also SJ302.1, SJ304.1; no longer X301.3
- net CONF0: now also R311.2; no longer R308.2
- net CONF1: now also R312.2; no longer R309.2
- net CONF2: now also R313.2; no longer R310.2
- net CONF3: now also R314.2; no longer R311.2
- net D0: now also R107.2; no longer R105.2
- net D1: now also R108.2; no longer R106.2
- net D10: now also R117.2; no longer R115.2
- net D11: now also R118.2; no longer R116.2
- net D12: now also R119.2; no longer R117.2
- net D13: now also R120.2; no longer R118.2
- net D14: now also R121.2; no longer R119.2
- net D15: now also R122.2; no longer R120.2
- net D2: now also R109.2; no longer R107.2
- net D3: now also R110.2; no longer R108.2
- net D4: now also R111.2; no longer R109.2
- net D5: now also R112.2; no longer R110.2
- net D6: now also R113.2; no longer R111.2
- net D7: now also R114.2; no longer R112.2
- net D8: now also R115.2; no longer R113.2
- net D9: now also R116.2; no longer R114.2
- net GND: now also C104.2, C106.-, R121.1, R122.1, R312.1, R313.1, R314.1; no longer C1.2, C104.-, R105.1, R106.1, R308.1, R309.1, R310.1
- net N$10: now also R308.2; no longer R312.2
- net N$7: now also R309.2; no longer R313.2
- net N$9: now also R310.2; no longer R314.2
- net STATUS0: now also R310.1; no longer R314.1
- net STATUS1: now also R309.1; no longer R313.1
- net STATUS2: now also R308.1; no longer R312.1
Routing:
- net !HALT: track 77.9 -> 174.0 mm, vias 3 -> 4
- net !RESET: track 232.8 -> 322.1 mm
- net COM0_TX_PIN: track 0.00 -> 35.4 mm
- net COM0_RX_PIN: track 0.00 -> 32.8 mm
- net COM0_RTS_PIN: track 0.00 -> 29.9 mm
- net COM0_CTS_PIN: track 0.00 -> 20.8 mm
- net COM0_RTS: track 15.6 -> 34.0 mm, vias 0 -> 1
- net COM0_CTS: track 24.2 -> 39.9 mm, vias 0 -> 2
- net COM0_RX: track 21.1 -> 36.2 mm
- net +5V: track 570.5 -> 577.9 mm
- net N$19: track 0.00 -> 2.90 mm
- net N$18: track 0.00 -> 2.90 mm
- net A_RX: track 120.8 -> 118.0 mm
- net A_TX: track 116.6 -> 113.8 mm
- net !A_RTS: track 118.7 -> 116.1 mm
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Other:
- board text added: "2019 Tristan Seifert"
- board text added: "JLCJLCJLCJLC"
- board text removed: "(c) 2019 Tristan Seifert"
