File: cpu-68000/ram-2mb.sch (EAGLE design)
At the start: 72 parts, among them IC101 74HC245DW, IC102 74HC245DW, IC103 74HC245DW, IC104 74HC245DW, IC105 74HC138D, IC106 GAL22V10D, IC107 74HC243D

Commit message: IO board: 	- Added 82C55 PIO
RAM board:
	- Tweaked tolerances between some traces
	- Fixed naming of parts
Parts:
- removed C116: 100nF, rcl:C-EUC0805
- added C103: 10µF, rcl:CPOL-EUSMCB
- C102: value 1µF -> 100nF; MOUSER 710-885012207078 -> 710-885012207072
- C104: value 120µF -> 100nF; device rcl:CPOL-EUE2.5-7 -> rcl:C-EUC0805; MOUSER 710-860020373007 -> 710-885012207072
- C105: value 10µF -> 100nF; device rcl:CPOL-EUSMCB -> rcl:C-EUC0805; MOUSER 581-TAJB106K020RNJV -> 710-885012207072
- C106: value 100nF -> 10µF; device rcl:C-EUC0805 -> rcl:CPOL-EUSMCB; MOUSER 710-885012207072 -> 581-TAJB106K020RNJV
- C108: value 10µF -> 1µF; device rcl:CPOL-EUSMCB -> rcl:C-EUC0805; MOUSER 581-TAJB106K020RNJV -> 710-885012207078
- C109: value 100nF -> 120µF; device rcl:C-EUC0805 -> rcl:CPOL-EUE2.5-7; MOUSER 710-885012207072 -> 710-860020373007
- IC105: value 74HC138D -> 74HC243D; device 74xx-eu:74HC138D -> 74xx-eu:74HC243D; MOUSER 595-SN74HC138DG4 -> 595-CD74HC243M96
- IC106: value GAL22V10D -> 74HC138D; device 68komputer:GAL22V10DIP24 -> 74xx-eu:74HC138D; MOUSER (none) -> 595-SN74HC138DG4; MOUSER_SOCKET 575-1104732441001000 -> (none)
- IC107: value 74HC243D -> GAL22V10D; device 74xx-eu:74HC243D -> 68komputer:GAL22V10DIP24; MOUSER 595-CD74HC243M96 -> (none); MOUSER_SOCKET (none) -> 575-1104732441001000
- R101: value 10k -> 3k; MOUSER 652-CR0805FX-1002ELF -> 652-CR0805JW-302ELF
- R103: value 3k -> 10k; MOUSER 652-CR0805JW-302ELF -> 652-CR0805FX-1002ELF
- renumbered S1 to S101
Connections:
- net !AS: now also IC107.IN5; no longer IC106.IN5
- net !CS: now also IC105A.GAB, IC106A.G2A, IC107.IO14; no longer IC105A.G2A, IC106.IO14, IC107A.GAB
- net !DTACK: now also IC107.IO16; no longer IC106.IO16
- net !LDS: now also IC107.IN3; no longer IC106.IN3
- net !LOE: now also IC107.IO20; no longer IC106.IO20
- net !LWE: now also IC107.IO21; no longer IC106.IO21
- net !RAM_CS0: now also IC106A.Y0; no longer IC105A.Y0
- net !RAM_CS1: now also IC106A.Y1; no longer IC105A.Y1
- net !RAM_CS2: now also IC106A.Y2; no longer IC105A.Y2
- net !RAM_CS3: now also IC106A.Y3; no longer IC105A.Y3
- net !RAM_CS4: now also IC106A.Y4; no longer IC105A.Y4
- net !RAM_CS5: now also IC106A.Y5; no longer IC105A.Y5
- net !RAM_CS6: now also IC106A.Y6; no longer IC105A.Y6
- net !RAM_CS7: now also IC106A.Y7; no longer IC105A.Y7
- net !RD: now also IC107.IO15; no longer IC106.IO15
- net !RESET: now also IC107.IN1/CLK; no longer IC106.IN1/CLK
- net !UDS: now also IC107.IN4; no longer IC106.IN4
- net !UOE: now also IC107.IO22; no longer IC106.IO22
- net !UWE: now also IC107.IO23; no longer IC106.IO23
- net +5V: now also C103.+, C104.1, C105.1, C106.+, C108.1, C109.+, IC105A.GBA, IC106A.G1, IC106P.VCC, IC107.VCC, R101.1; no longer C104.+, C105.+, C106.1, C108.+, C109.1, C116.1, IC105A.G1, IC106.VCC, IC107A.GBA, IC107P.VCC, R103.1
- net A17: now also IC105A.A1; no longer IC107A.A1
- net A18: now also IC106A.A; no longer IC105A.A
- net A19: now also IC106A.B, IC107.IN6; no longer IC105A.B, IC106.IN6
- net A20: now also IC106A.C, IC107.IN7; no longer IC105A.C, IC106.IN7
- net A21: now also IC107.IN8; no longer IC106.IN8
- net A22: now also IC107.IN9; no longer IC106.IN9
- net A23: now also IC107.IN13; no longer IC106.IN13
- net ADDR_SET0: now also IC107.IN10, R103.1; no longer IC106.IN10, R102.1
- net ADDR_SET1: now also IC107.IN11, R102.1; no longer IC106.IN11, R101.1
- net GND: now also C103.-, C104.2, C105.2, C106.-, C108.2, C109.-, IC105A.A2, IC105A.A3, IC105A.A4, IC106A.G2B, IC106P.GND, IC107.GND, R103.2; no longer C104.-, C105.-, C106.2, C108.-, C109.2, C116.2, IC105A.G2B, IC106.GND, IC107A.A2, IC107A.A3, IC107A.A4, IC107P.GND, R101.2
- net N$18: now also R101.2; no longer R103.2
- net N$5: now also IC107.IO19; no longer IC106.IO19
- net N$6: now also IC107.IO18; no longer IC106.IO18
- net N$7: now also IC107.IO17; no longer IC106.IO17
- net R/!W!: now also IC107.IN2; no longer IC106.IN2
- net RAM_A16: now also IC105A.B1; no longer IC107A.B1
Other:
- moved on the sheet: C101, C102, C107, C110, C111, C112, IC105P, R101, R102, R103

Commit message: Rev01 of CPU-68000 and 2MB SRAM board sent to production
Parts:
- added LED102: (no value), led:LEDCHIPLED_1206
- added R104: 3k, rcl:R-EU_R2012
Connections:
- removed net N$5: IC107.IO19
- removed net N$6: IC107.IO18
- removed net N$7: IC107.IO17
- new net !CS_LED: IC105A.B2, LED102.C
- new net N$1: LED102.A, R104.2
- net !CS: now also IC105A.A2; no longer IC103A.G, IC104A.G, IC105A.GAB
- net +5V: now also R104.1; no longer IC105A.GBA
- net GND: now also IC103A.G, IC104A.G, IC105A.GAB, IC105A.GBA; no longer IC105A.A2
Changed lines of the file:
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@@
 <attribute name="MOUSER" value="710-885012207072"/>
 </part>
-<part name="P+12" library="supply1" library_urn="urn:adsk.eagle:library:371" deviceset="+5V" device=""/>
 <part name="GND11" library="supply1" library_urn="urn:adsk.eagle:library:371" deviceset="GND" device=""/>
 <part name="GND7" library="supply1" library_urn="urn:adsk.eagle:library:371" deviceset="GND" device=""/>
+<part name="GND12" library="supply1" library_urn="urn:adsk.eagle:library:371" deviceset="GND" device=""/>
+<part name="GND13" library="supply1" library_urn="urn:adsk.eagle:library:371" deviceset="GND" device=""/>
+<part name="GND14" library="supply1" library_urn="urn:adsk.eagle:library:371" deviceset="GND" device=""/>
+<part name="R104" library="rcl" library_urn="urn:adsk.eagle:library:334" deviceset="R-EU_" device="R2012" package3d_urn="urn:adsk.eagle:package:23543/2" value="3k">
+<attribute name="MOUSER" value="652-CR0805JW-302ELF"/>
+</part>
+<part name="LED102" library="led" library_urn="urn:adsk.eagle:library:259" deviceset="LED" device="CHIPLED_1206" package3d_urn="urn:adsk.eagle:package:15823/2">
+<attribute name="MOUSER" value="710-156120VS75300"/>
+</part>
+<part name="P+11" library="supply1" library_urn="urn:adsk.eagle:library:371" deviceset="+5V" device=""/>
 </parts>
 <sheets>
@@
 <attribute name="NAME" x="62.865" y="60.325" size="1.778" layer="95"/>
 </instance>
-<instance part="P+12" gate="1" x="121.92" y="124.46" smashed="yes" rot="R90">
-<attribute name="VALUE" x="121.92" y="124.46" size="1.778" layer="96" rot="R180"/>
-</instance>
 <instance part="GND11" gate="1" x="121.92" y="132.08" smashed="yes" rot="R270">
 <attribute name="VALUE" x="119.38" y="134.62" size="1.778" layer="96" rot="R270"/>
@@
 <instance part="GND7" gate="1" x="129.54" y="96.52" smashed="yes">
 <attribute name="VALUE" x="127" y="93.98" size="1.778" layer="96"/>
+</instance>
+<instance part="GND12" gate="1" x="71.12" y="106.68" smashed="yes">
+<attribute name="VALUE" x="68.58" y="104.14" size="1.778" layer="96"/>
+</instance>
+<instance part="GND13" gate="1" x="71.12" y="147.32" smashed="yes">
+<attribute name="VALUE" x="68.58" y="144.78" size="1.778" layer="96"/>
+</instance>
+<instance part="GND14" gate="1" x="124.46" y="121.92" smashed="yes">
+<attribute name="VALUE" x="121.92" y="119.38" size="1.778" layer="96"/>
+</instance>
+<instance part="R104" gate="G$1" x="220.98" y="71.12" smashed="yes" rot="R180">
+<attribute name="NAME" x="224.79" y="69.6214" size="1.778" layer="95" rot="R180"/>
+<attribute name="VALUE" x="224.79" y="74.422" size="1.778" layer="96" rot="R180"/>
+<attribute name="MOUSER" x="220.98" y="71.12" size="1.778" layer="96" rot="R180" align="top-left" display="off"/>
+</instance>
+<instance part="LED102" gate="G$1" x="213.36" y="71.12" smashed="yes" rot="R270">
+<attribute name="NAME" x="208.788" y="67.564" size="1.778" layer="95"/>
+<attribute name="VALUE" x="208.788" y="65.405" size="1.778" layer="96"/>
+<attribute name="MOUSER" x="213.36" y="71.12" size="1.778" layer="96" rot="R270" align="top-left" display="off"/>
+</instance>
+<instance part="P+11" gate="1" x="228.6" y="71.12" smashed="yes" rot="R270">
+<attribute name="VALUE" x="231.14" y="71.12" size="1.778" layer="96"/>
 </instance>
 </instances>
@@
 </segment>
 </bus>
-<bus name="RAM_A[0..16],!RAM_CS[0..7]">
+<bus name="!CS_LED,RAM_A[0..16],!RAM_CS[0..7]">
 <segment>
 <wire x1="160.02" y1="177.8" x2="160.02" y2="119.38" width="0.762" layer="92"/>
-<label x="162.56" y="144.78" size="1.778" layer="95" rot="R90"/>
+<label x="162.56" y="137.16" size="1.778" layer="95" rot="R90"/>
 </segment>
 </bus>
@@
 </segment>
 <segment>
-<pinref part="IC105" gate="A" pin="GBA"/>
-<pinref part="P+12" gate="1" pin="+5V"/>
+<pinref part="R104" gate="G$1" pin="1"/>
+<pinref part="P+11" gate="1" pin="+5V"/>
+<junction x="226.06" y="71.12"/>
 </segment>
 </net>
@@
 <segment>
 <pinref part="IC105" gate="A" pin="A4"/>
-<pinref part="IC105" gate="A" pin="A2"/>
 <wire x1="124.46" y1="132.08" x2="124.46" y2="134.62" width="0.1524" layer="91"/>
 <pinref part="IC105" gate="A" pin="A3"/>
-<wire x1="124.46" y1="134.62" x2="124.46" y2="137.16" width="0.1524" layer="91"/>
-<junction x="124.46" y="134.62"/>
 <pinref part="GND11" gate="1" pin="GND"/>
 <junction x="124.46" y="132.08"/>
@@
 <junction x="129.54" y="99.06"/>
 </segment>
+<segment>
+<pinref part="IC104" gate="A" pin="G"/>
+<pinref part="GND12" gate="1" pin="GND"/>
+</segment>
+<segment>
+<pinref part="IC103" gate="A" pin="G"/>
+<pinref part="GND13" gate="1" pin="GND"/>
+</segment>
+<segment>
+<pinref part="IC105" gate="A" pin="GBA"/>
+<pinref part="IC105" gate="A" pin="GAB"/>
+<wire x1="124.46" y1="124.46" x2="124.46" y2="127" width="0.1524" layer="91"/>
+<pinref part="GND14" gate="1" pin="GND"/>
+<junction x="124.46" y="124.46"/>
+</segment>
 </net>
 <net name="!BG" class="0">
@@
 </segment>
 <segment>
-<pinref part="IC103" gate="A" pin="G"/>
-<wire x1="71.12" y1="149.86" x2="66.04" y2="149.86" width="0.1524" layer="91"/>
-<wire x1="66.04" y1="149.86" x2="63.5" y2="147.32" width="0.1524" layer="91"/>
-</segment>
-<segment>
-<pinref part="IC104" gate="A" pin="G"/>
-<wire x1="71.12" y1="109.22" x2="66.04" y2="109.22" width="0.1524" layer="91"/>
-<wire x1="66.04" y1="109.22" x2="63.5" y2="106.68" width="0.1524" layer="91"/>
-</segment>
-<segment>
 <pinref part="IC107" gate="G$1" pin="IO14"/>
 <wire x1="220.98" y1="175.26" x2="226.06" y2="175.26" width="0.1524" layer="91"/>
@@
 </segment>
 <segment>
-<pinref part="IC105" gate="A" pin="GAB"/>
-<wire x1="124.46" y1="127" x2="119.38" y2="127" width="0.1524" layer="91"/>
-<wire x1="119.38" y1="127" x2="116.84" y2="124.46" width="0.1524" layer="91"/>
+<pinref part="IC105" gate="A" pin="A2"/>
+<wire x1="124.46" y1="137.16" x2="119.38" y2="137.16" width="0.1524" layer="91"/>
+<wire x1="119.38" y1="137.16" x2="116.84" y2="134.62" width="0.1524" layer="91"/>
 </segment>
 </net>
@@
 </segment>
 </net>
-<net name="N$5" class="0">
-<segment>
-<pinref part="IC107" gate="G$1" pin="IO19"/>
-<wire x1="220.98" y1="162.56" x2="226.06" y2="162.56" width="0.1524" layer="91"/>
-</segment>
-</net>
-<net name="N$6" class="0">
-<segment>
-<pinref part="IC107" gate="G$1" pin="IO18"/>
-<wire x1="220.98" y1="165.1" x2="226.06" y2="165.1" width="0.1524" layer="91"/>
-</segment>
-</net>
-<net name="N$7" class="0">
-<segment>
-<pinref part="IC107" gate="G$1" pin="IO17"/>
-<wire x1="220.98" y1="167.64" x2="226.06" y2="167.64" width="0.1524" layer="91"/>
-</segment>
-</net>
 <net name="N$18" class="0">
 <segment>
@@
 </segment>
 </net>
+<net name="!CS_LED" class="0">
+<segment>
+<pinref part="IC105" gate="A" pin="B2"/>
+<wire x1="149.86" y1="137.16" x2="157.48" y2="137.16" width="0.1524" layer="91"/>
+<wire x1="157.48" y1="137.16" x2="160.02" y2="134.62" width="0.1524" layer="91"/>
+</segment>
+<segment>
+<pinref part="LED102" gate="G$1" pin="C"/>
+<wire x1="208.28" y1="71.12" x2="203.2" y2="71.12" width="0.1524" layer="91"/>
+<label x="203.2" y="71.12" size="1.778" layer="95" rot="R180" xref="yes"/>
+</segment>
+</net>
+<net name="N$1" class="0">
+<segment>
+<pinref part="R104" gate="G$1" pin="2"/>
+<pinref part="LED102" gate="G$1" pin="A"/>
+<junction x="215.9" y="71.12"/>
+</segment>
+</net>
