File: cpu-68000/sound.brd (EAGLE design)
At the start: 160 x 100 mm, 26 parts, among them IC101 74HC245DW, IC2 IDT7006

Commit message: Added sound CPU RAM, LED indicators, MIDI UART
Parts:
- removed LED101: (no value), led:CHIPLED_1206
- removed R101: 3k, rcl:R2012
- added C10, C12, C13, C401, C402, C403, C8: 100nF, rcl:C0805
- added C11, C404: 10µF, rcl:SMC_B
- added C405, C406: 27pF, rcl:C0805
- added C9: 1µF, rcl:C0805
- added D401: 1N914, diode:DO35-10
- added IC3, IC4: 74HC04D, 74xx-eu:SO14
- added IC401: 74HCT14N, 74xx-eu:DIL14
- added IC402: SCC2691, 68komputer:DIL24S
- added IC5: IS61C5128AL, 68komputer:TSOP44-II
- added J401, J402: DIN5, SparkFun-Connectors:DIN5-RA-PTH
- added LED1, LED2, LED3, LED4: 555-4001, 68komputer:555-4001
- added OK401: H11L1M, optocoupler:DIL06
- added Q401: 3MHz, crystal:HC49/S
- added R1, R10, R11, R12, R13, R14, R15, R16, R2, R3, R4, R5, R6, R7, R8, R9: 2k7, rcl:R2012
- added R401, R406: 220R, rcl:R2012
- added R402, R407: 4k7, rcl:R2012
- moved IC1 8.00 mm to (138.5, 76.5), turned to 90 degrees
Connections:
- removed net N$18: LED101.A, R101.2
- new net !BUS_MBOX_IRQ: IC3.1
- new net !CPU_MBOX_IRQ: IC4.3
- new net !CPU_OE: IC5.37
- new net !CPU_RAM_CS: IC5.8
- new net !MIDI_IRQ: IC4.1, IC402.13, R407.1
- new net !MIDI_UART_CS: IC402.14
- new net !RD: IC402.1
- new net !YM3812_IRQ: IC4.9
- new net APERTURE_BANK: IC3.5
- new net LED_APERTURE_BANK: IC3.8, R3.2
- new net LED_BR: IC3.4, R4.2
- new net LED_BUS_MBOX_IRQ: IC3.2, R2.2
- new net LED_CPU_BG: IC4.6, R7.2
- new net LED_CPU_HALT: IC3.12, R6.2
- new net LED_CPU_MBOX_IRQ: IC4.4, R8.2
- new net LED_CPU_RESET: IC3.10, R5.2
- new net LED_MIDI_IRQ: IC4.2, R10.2
- new net LED_MIDI_RX: IC4.10, R11.2
- new net LED_MIDI_TX: IC4.12, R12.2
- new net LED_STATUS_0: R13.2
- new net LED_STATUS_1: R14.2
- new net LED_STATUS_2: R15.2
- new net LED_STATUS_3: R16.2
- new net LED_YM3812_IRQ: IC4.8, R9.2
- new net MIDI_RESET: IC401.8, IC402.11
- new net MIDI_RX: IC4.11, IC402.2, OK401.4, R402.1
- new net MIDI_RX_+: D401.A, J401.5, OK401.2
- new net MIDI_RX_-: D401.C, OK401.1, R401.2
- new net MIDI_TX: IC4.13, IC401.13, IC402.3
- new net MIDI_TX_-: IC401.10, J402.5
- new net MIDI_UART_X1: C405.2, IC402.9, Q401.1
- new net MIDI_UART_X2: C406.2, IC402.10, Q401.2
- new net N$10: IC3.6, IC3.9
- new net N$11: LED2.A2, R7.1
- new net N$12: LED2.A1, R8.1
- new net N$13: LED3.A4, R9.1
- new net N$14: J401.4, R401.1
- new net N$15: LED3.A3, R10.1
- new net N$16: IC401.11, IC401.12
- new net N$17: J402.4, R406.1
- new net N$19: LED3.A2, R11.1
- new net N$2: LED1.A4, R1.1
- new net N$20: LED3.A1, R12.1
- new net N$21: LED4.A4, R13.1
- new net N$22: LED4.A3, R14.1
- new net N$23: LED4.A2, R15.1
- new net N$24: LED4.A1, R16.1
- new net N$4: LED1.A3, R2.1
- new net N$5: LED1.A2, R3.1
- new net N$6: LED1.A1, R4.1
- new net N$7: LED2.A4, R5.1
- new net N$9: LED2.A3, R6.1
- net !CPU_BG: now also IC4.5
- net !CPU_BR: now also IC3.3
- net !CPU_HALT: now also IC3.13
- net !CPU_RESET: now also IC3.11, IC401.9
- net +5V: now also C10.1, C11.+, C12.1, C13.1, C401.1, C402.1, C403.1, C404.+, C8.1, C9.1, IC3.14, IC4.14, IC401.14, IC402.24, IC5.11, IC5.33, OK401.6, R1.2, R402.2, R406.2, R407.2; no longer R101.1
- net CPU_A0: now also IC402.8, IC5.3
- net CPU_A1: now also IC402.7, IC5.4
- net CPU_A10: now also IC5.26
- net CPU_A11: now also IC5.27
- net CPU_A12: now also IC5.28
- net CPU_A13: now also IC5.29
- net CPU_A14: now also IC5.30
- net CPU_A15: now also IC5.38
- net CPU_A16: now also IC5.39
- net CPU_A17: now also IC5.40
- net CPU_A18: now also IC5.41
- net CPU_A2: now also IC402.6, IC5.5
- net CPU_A3: now also IC5.6
- net CPU_A4: now also IC5.7
- net CPU_A5: now also IC5.16
- net CPU_A6: now also IC5.17
- net CPU_A7: now also IC5.18
- net CPU_A8: now also IC5.19
- net CPU_A9: now also IC5.20
- net CPU_D0: now also IC402.22, IC5.9
- net CPU_D1: now also IC402.21, IC5.10
- net CPU_D2: now also IC402.20, IC5.13
- net CPU_D3: now also IC402.19, IC5.14
- net CPU_D4: now also IC402.18, IC5.31
- net CPU_D5: now also IC402.17, IC5.32
- net CPU_D6: now also IC402.16, IC5.35
- net CPU_D7: now also IC402.15, IC5.36
- net CPU_R/!W!: now also IC402.23, IC5.15
- net GND: now also C10.2, C11.-, C12.2, C13.2, C401.2, C402.2, C403.2, C404.-, C405.1, C406.1, C8.2, C9.2, IC3.7, IC4.7, IC401.1, IC401.3, IC401.5, IC401.7, IC402.12, IC5.12, IC5.34, J402.2, LED1.K1, LED1.K2, LED1.K3, LED1.K4, LED2.K1, LED2.K2, LED2.K3, LED2.K4, LED3.K1, LED3.K2, LED3.K3, LED3.K4, LED4.K1, LED4.K2, LED4.K3, LED4.K4, OK401.5; no longer LED101.C
