File: cpu-68000/sound.sch (EAGLE design)
At the start: 26 parts, among them IC101 74HC245DW, IC2 IDT7006

Commit message: Added sound CPU RAM, LED indicators, MIDI UART
Parts:
- removed LED101: (no value), led:LEDCHIPLED_1206
- removed R101: 3k, rcl:R-EU_R2012
- added C10, C12, C13, C401, C402, C403, C8: 100nF, rcl:C-EUC0805
- added C11, C404: 10µF, rcl:CPOL-EUSMCB
- added C405, C406: 27pF, rcl:C-EUC0805
- added C9: 1µF, rcl:C-EUC0805
- added D401: 1N914, diode:1N4148DO35-10
- added IC3, IC4: 74HC04D, 74xx-eu:74HC04D
- added IC401: 74HCT14N, 74xx-eu:74HCT14N
- added IC402: SCC2691, 68komputer:SCC2691
- added IC5: IS61C5128AL, 68komputer:IS61C5128AL
- added J401, J402: DIN5, SparkFun-Connectors:DIN5
- added LED1, LED2, LED3, LED4: 555-4001, 68komputer:555-4001
- added OK401: H11L1M, optocoupler:H11L1M
- added Q401: 3MHz, crystal:CRYSTALHC49S
- added R1, R10, R11, R12, R13, R14, R15, R16, R2, R3, R4, R5, R6, R7, R8, R9: 2k7, rcl:R-EU_R2012
- added R401, R406: 220R, rcl:R-EU_R2012
- added R402, R407: 4k7, rcl:R-EU_R2012
Connections:
- removed net N$18: LED101.A, R101.2
- new net !BUS_MBOX_IRQ: IC3A.I
- new net !CPU_MBOX_IRQ: IC4B.I
- new net !CPU_OE: IC5.!OE
- new net !CPU_RAM_CS: IC5.!CS
- new net !MIDI_IRQ: IC402.!IRQ, IC4A.I, R407.1
- new net !MIDI_UART_CS: IC402.!CS
- new net !RD: IC402.!RD
- new net !YM3812_IRQ: IC4D.I
- new net APERTURE_BANK: IC3C.I
- new net LED_APERTURE_BANK: IC3D.O, R3.2
- new net LED_BR: IC3B.O, R4.2
- new net LED_BUS_MBOX_IRQ: IC3A.O, R2.2
- new net LED_CPU_BG: IC4C.O, R7.2
- new net LED_CPU_HALT: IC3F.O, R6.2
- new net LED_CPU_MBOX_IRQ: IC4B.O, R8.2
- new net LED_CPU_RESET: IC3E.O, R5.2
- new net LED_MIDI_IRQ: IC4A.O, R10.2
- new net LED_MIDI_RX: IC4E.O, R11.2
- new net LED_MIDI_TX: IC4F.O, R12.2
- new net LED_STATUS_0: R13.2
- new net LED_STATUS_1: R14.2
- new net LED_STATUS_2: R15.2
- new net LED_STATUS_3: R16.2
- new net LED_YM3812_IRQ: IC4D.O, R9.2
- new net MIDI_RESET: IC401C.O, IC402.RESET
- new net MIDI_RX: IC402.RXD, IC4E.I, OK401.OUT, R402.1
- new net MIDI_RX_+: D401.A, J401.5, OK401.C
- new net MIDI_RX_-: D401.C, OK401.A, R401.2
- new net MIDI_TX: IC401A.I, IC402.TXD, IC4F.I
- new net MIDI_TX_-: IC401B.O, J402.5
- new net MIDI_UART_X1: C405.2, IC402.X1/CLK, Q401.1
- new net MIDI_UART_X2: C406.2, IC402.X2, Q401.2
- new net N$10: IC3C.O, IC3D.I
- new net N$11: LED2.A2, R7.1
- new net N$12: LED2.A1, R8.1
- new net N$13: LED3.A4, R9.1
- new net N$14: J401.4, R401.1
- new net N$15: LED3.A3, R10.1
- new net N$16: IC401A.O, IC401B.I
- new net N$17: J402.4, R406.1
- new net N$19: LED3.A2, R11.1
- new net N$2: LED1.A4, R1.1
- new net N$20: LED3.A1, R12.1
- new net N$21: LED4.A4, R13.1
- new net N$22: LED4.A3, R14.1
- new net N$23: LED4.A2, R15.1
- new net N$24: LED4.A1, R16.1
- new net N$4: LED1.A3, R2.1
- new net N$5: LED1.A2, R3.1
- new net N$6: LED1.A1, R4.1
- new net N$7: LED2.A4, R5.1
- new net N$9: LED2.A3, R6.1
- net !CPU_BG: now also IC4C.I
- net !CPU_BR: now also IC3B.I
- net !CPU_HALT: now also IC3F.I
- net !CPU_RESET: now also IC3E.I, IC401C.I
- net +5V: now also C10.1, C11.+, C12.1, C13.1, C401.1, C402.1, C403.1, C404.+, C8.1, C9.1, IC3P.VCC, IC401P.VCC, IC402.VCC, IC4P.VCC, IC5.VCC, OK401.VCC, R1.2, R402.2, R406.2, R407.2; no longer R101.1
- net CPU_A0: now also IC402.A0, IC5.A0
- net CPU_A1: now also IC402.A1, IC5.A1
- net CPU_A10: now also IC5.A10
- net CPU_A11: now also IC5.A11
- net CPU_A12: now also IC5.A12
- net CPU_A13: now also IC5.A13
- net CPU_A14: now also IC5.A14
- net CPU_A15: now also IC5.A15
- net CPU_A16: now also IC5.A16
- net CPU_A17: now also IC5.A17
- net CPU_A18: now also IC5.A18
- net CPU_A2: now also IC402.A2, IC5.A2
- net CPU_A3: now also IC5.A3
- net CPU_A4: now also IC5.A4
- net CPU_A5: now also IC5.A5
- net CPU_A6: now also IC5.A6
- net CPU_A7: now also IC5.A7
- net CPU_A8: now also IC5.A8
- net CPU_A9: now also IC5.A9
- net CPU_D0: now also IC402.D0, IC5.D0
- net CPU_D1: now also IC402.D1, IC5.D1
- net CPU_D2: now also IC402.D2, IC5.D2
- net CPU_D3: now also IC402.D3, IC5.D3
- net CPU_D4: now also IC402.D4, IC5.D4
- net CPU_D5: now also IC402.D5, IC5.D5
- net CPU_D6: now also IC402.D6, IC5.D6
- net CPU_D7: now also IC402.D7, IC5.D7
- net CPU_R/!W!: now also IC402.!WR, IC5.!WE
- net GND: now also C10.2, C11.-, C12.2, C13.2, C401.2, C402.2, C403.2, C404.-, C405.1, C406.1, C8.2, C9.2, IC3P.GND, IC401D.I, IC401E.I, IC401F.I, IC401P.GND, IC402.GND, IC4P.GND, IC5.GND, J402.2, LED1.K1, LED1.K2, LED1.K3, LED1.K4, LED2.K1, LED2.K2, LED2.K3, LED2.K4, LED3.K1, LED3.K2, LED3.K3, LED3.K4, LED4.K1, LED4.K2, LED4.K3, LED4.K4, OK401.GND; no longer LED101.C
