File: cpu-68000/cpu-68000.kicad_sch (KiCad schematic)
At the start: 14 parts, among them J101 Conn_02x04_Odd_Even, U101 ATF22V10C, U102 ATF22V10C, U103 74HC175, U104 74HC05, X101 10MHz

Commit message: Minor cleanup of CPU board
- Switched out of stock 2 bit level shifters for 8 bit part we already
  have; this means that the function codes will be buffered along with
  all other signals.
Connections:
- net GND: now also U104.3
- net EXT_MEM: no longer names the net of U102.15 (IO2)
- net EXT_MEM: no longer U104.3
- net ~{EXT_MEM}: no longer names the net of U104.4
Other:
- sheet Backplane Connection ports: added none; removed ~{MEM}
- sheet Memory ports: added none; removed ~{LDS}, ~{UDS}
- sheet Peripherals ports: added none; removed ~{RD}
- note removed: "~{EXT_MEM} asserted when access is memory space"
Changed lines of the file:
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@@
-    (stroke (width 0) (type default) (color 0 0 0 0))
-  )
-  (wire (pts (xy 101.6 59.055) (xy 89.535 59.055))
     (stroke (width 0) (type default) (color 0 0 0 0))
   )
@@
     (stroke (width 0) (type default) (color 0 0 0 0))
   )
-  (wire (pts (xy 189.23 24.13) (xy 177.8 24.13))
-    (stroke (width 0) (type default) (color 0 0 0 0))
-  )
   (wire (pts (xy 146.685 151.13) (xy 134.62 151.13))
     (stroke (width 0) (type default) (color 0 0 0 0))
@@
     (stroke (width 0) (type default) (color 0 0 0 0))
   )
-  (wire (pts (xy 161.925 122.555) (xy 172.085 122.555))
-    (stroke (width 0) (type default) (color 0 0 0 0))
-  )
   (wire (pts (xy 55.88 93.345) (xy 67.945 93.345))
     (stroke (width 0) (type default) (color 0 0 0 0))
@@
     (stroke (width 0) (type default) (color 0 0 0 0))
   )
-  (wire (pts (xy 55.88 140.97) (xy 67.945 140.97))
-    (stroke (width 0) (type default) (color 0 0 0 0))
-  )
   (wire (pts (xy 114.935 130.81) (xy 86.995 130.81))
     (stroke (width 0) (type default) (color 0 0 0 0))
@@
     (stroke (width 0) (type default) (color 0 0 0 0))
   )
-  (wire (pts (xy 242.57 66.675) (xy 254 66.675))
-    (stroke (width 0) (type default) (color 0 0 0 0))
-  )
   (wire (pts (xy 84.455 128.27) (xy 84.455 158.75))
     (stroke (width 0) (type default) (color 0 0 0 0))
@@
     (stroke (width 0) (type default) (color 0 0 0 0))
   )
-  (wire (pts (xy 134.62 122.555) (xy 146.685 122.555))
-    (stroke (width 0) (type default) (color 0 0 0 0))
-  )
   (wire (pts (xy 242.57 79.375) (xy 254 79.375))
     (stroke (width 0) (type default) (color 0 0 0 0))
@@
   )
   (wire (pts (xy 89.535 48.895) (xy 101.6 48.895))
-    (stroke (width 0) (type default) (color 0 0 0 0))
-  )
-  (wire (pts (xy 189.23 21.59) (xy 177.8 21.59))
     (stroke (width 0) (type default) (color 0 0 0 0))
   )
@@
     (effects (font (size 1.27 1.27)) (justify left bottom))
   )
-  (text "~{EXT_MEM} asserted when access is memory space" (at 135.255 113.03 0)
-    (effects (font (size 1.27 1.27)) (justify left bottom))
-  )
   (text "DTACK_FAST / DTACK_SLOW asserted for RAM/ROM and peripherals respectively"
     (at 15.24 196.85 0)
@@
     (effects (font (size 1.27 1.27)) (justify left bottom))
   )
-  (label "EXT_MEM" (at 67.945 140.97 180)
-    (effects (font (size 1.27 1.27)) (justify right bottom))
-  )
   (label "~{BG}" (at 23.495 88.265 0)
     (effects (font (size 1.27 1.27)) (justify left bottom))
@@
     (effects (font (size 1.27 1.27)) (justify left bottom))
   )
-  (label "~{UDS}" (at 189.23 21.59 180)
-    (effects (font (size 1.27 1.27)) (justify right bottom))
-  )
   (label "A[1..23]" (at 189.23 33.655 180)
     (effects (font (size 1.27 1.27)) (justify right bottom))
@@
     (effects (font (size 1.27 1.27)) (justify left bottom))
   )
-  (label "~{LDS}" (at 189.23 24.13 180)
-    (effects (font (size 1.27 1.27)) (justify right bottom))
-  )
   (label "~{BG}" (at 240.03 24.13 180)
     (effects (font (size 1.27 1.27)) (justify right bottom))
@@
     (effects (font (size 1.27 1.27)) (justify left bottom))
   )
-  (label "~{RD}" (at 89.535 59.055 0)
-    (effects (font (size 1.27 1.27)) (justify left bottom))
-  )
   (label "~{IACK_DUART}" (at 191.77 92.71 0)
     (effects (font (size 1.27 1.27)) (justify left bottom))
@@
     (effects (font (size 1.27 1.27)) (justify left bottom))
   )
-  (label "~{EXT_MEM}" (at 172.085 122.555 180)
-    (effects (font (size 1.27 1.27)) (justify right bottom))
-  )
   (label "~{IRQ_DUART}" (at 191.77 87.63 0)
     (effects (font (size 1.27 1.27)) (justify left bottom))
@@
     (effects (font (size 1.27 1.27)) (justify left bottom))
   )
-  (label "~{EXT_MEM}" (at 242.57 66.675 0)
-    (effects (font (size 1.27 1.27)) (justify left bottom))
-  )
   (label "~{BR}" (at 242.57 34.29 0)
     (effects (font (size 1.27 1.27)) (justify left bottom))
@@
   (label "DTACK_FAST" (at 67.945 156.21 180)
     (effects (font (size 1.27 1.27)) (justify right bottom))
-  )
-  (label "EXT_MEM" (at 134.62 122.555 0)
-    (effects (font (size 1.27 1.27)) (justify left bottom))
   )
   (label "CLK" (at 241.3 150.495 0)
@@
     (pin "1")
   )
+  (symbol (lib_id "power:GND") (at 146.685 122.555 0) (unit 1)
+    (in_bom yes) (on_board yes) (fields_autoplaced)
+    (property "Reference" "#PWR0235" (id 0) (at 146.685 128.905 0)
+      (effects (font (size 1.27 1.27)) hide)
+    )
+    (property "Value" "GND" (id 1) (at 146.685 127.1175 0))
+    (property "Footprint" "" (id 2) (at 146.685 122.555 0)
+      (effects (font (size 1.27 1.27)) hide)
+    )
+    (property "Datasheet" "" (id 3) (at 146.685 122.555 0)
+      (effects (font (size 1.27 1.27)) hide)
+    )
+    (pin "1")
+  )
   (symbol (lib_id "Device:C_Small") (at 139.7 174.625 0) (unit 1)
     (in_bom yes) (on_board yes) (fields_autoplaced)
@@
       (effects (font (size 1.27 1.27)) (justify left))
     )
-    (pin "~{RD}" input (at 101.6 59.055 180)
-      (effects (font (size 1.27 1.27)) (justify left))
-    )
     (pin "I2C_SCL" bidirectional (at 127 21.59 0)
       (effects (font (size 1.27 1.27)) (justify right))
@@
       (effects (font (size 1.27 1.27)) (justify left))
     )
-    (pin "~{MEM}" input (at 254 66.675 180)
-      (effects (font (size 1.27 1.27)) (justify left))
-    )
     (pin "~{I2C_BUS_IRQ}" output (at 254 49.53 180)
       (effects (font (size 1.27 1.27)) (justify left))
@@
     (property "Sheet file" "memory.kicad_sch" (id 1) (at 152.4 83.1346 0)
       (effects (font (size 1.27 1.27)) (justify left top))
-    )
-    (pin "~{UDS}" input (at 177.8 21.59 0)
-      (effects (font (size 1.27 1.27)) (justify right))
-    )
-    (pin "~{LDS}" input (at 177.8 24.13 0)
-      (effects (font (size 1.27 1.27)) (justify right))
     )
     (pin "D[0..15]" bidirectional (at 177.8 31.115 0)
@@
       (reference "#PWR0141") (unit 1) (value "GND") (footprint "")
     )
+    (path "/dd09b3c7-f3f1-4702-9c67-cfc029c2d128/7e607138-fa2c-4632-93b7-82e929c43652"
+      (reference "#PWR0142") (unit 1) (value "GND") (footprint "")
+    )
     (path "/a80fdcbe-0bb0-435d-8e84-e8399e2a8c71/b56470d6-5960-4d62-9665-9bfc99b9f0da"
       (reference "#PWR0143") (unit 1) (value "GND") (footprint "")
@@
       (reference "#PWR0225") (unit 1) (value "GND") (footprint "")
     )
+    (path "/dd09b3c7-f3f1-4702-9c67-cfc029c2d128/469917e8-5327-433c-acfc-b1c0428ab4fe"
+      (reference "#PWR0226") (unit 1) (value "GND") (footprint "")
+    )
+    (path "/dd09b3c7-f3f1-4702-9c67-cfc029c2d128/32d0f83c-4085-40fd-848b-7cf4838a4895"
+      (reference "#PWR0227") (unit 1) (value "+5V") (footprint "")
+    )
     (path "/a80fdcbe-0bb0-435d-8e84-e8399e2a8c71/6ba3879b-d4c4-4a67-affb-5eb32c80b592"
       (reference "#PWR0228") (unit 1) (value "+5V") (footprint "")
@@
       (reference "#PWR0232") (unit 1) (value "+5V") (footprint "")
     )
+    (path "/dd09b3c7-f3f1-4702-9c67-cfc029c2d128/fe99561b-aa95-4a36-97d7-9991ca2a84e3"
+      (reference "#PWR0233") (unit 1) (value "+5V") (footprint "")
+    )
+    (path "/dd09b3c7-f3f1-4702-9c67-cfc029c2d128/55c6a896-bc50-4f6e-8630-f9d93838f599"
+      (reference "#PWR0234") (unit 1) (value "GND") (footprint "")
+    )
+    (path "/9eea8331-9c75-4147-900e-277643181cc1"
+      (reference "#PWR0235") (unit 1) (value "GND") (footprint "")
+    )
     (path "/a80fdcbe-0bb0-435d-8e84-e8399e2a8c71/10697594-7c7d-434b-bdb6-30973b3c7203"
       (reference "#PWR0237") (unit 1) (value "GND") (footprint "")
     )
-    (path "/dd09b3c7-f3f1-4702-9c67-cfc029c2d128/58fa0c43-be9e-4077-8fd0-af5c69798796"
-      (reference "#PWR0241") (unit 1) (value "+5V") (footprint "")
-    )
-    (path "/dd09b3c7-f3f1-4702-9c67-cfc029c2d128/49b3deb9-059e-4fa2-b466-ec290389dd77"
-      (reference "#PWR0242") (unit 1) (value "+5V") (footprint "")
-    )
     (path "/dd09b3c7-f3f1-4702-9c67-cfc029c2d128/d5418365-e147-4269-9bc4-7cc70697b83f"
       (reference "#PWR0243") (unit 1) (value "+5V") (footprint "")
@@
       (reference "#PWR0244") (unit 1) (value "GND") (footprint "")
     )
-    (path "/dd09b3c7-f3f1-4702-9c67-cfc029c2d128/385922c8-1f72-4410-bf9e-616dbc1f31fb"
-      (reference "#PWR0245") (unit 1) (value "+5V") (footprint "")
-    )
-    (path "/dd09b3c7-f3f1-4702-9c67-cfc029c2d128/b76614ee-9a78-4f90-bf0f-45aa05155358"
-      (reference "#PWR0246") (unit 1) (value "GND") (footprint "")
-    )
-    (path "/dd09b3c7-f3f1-4702-9c67-cfc029c2d128/14fa2517-40cc-4dd1-ba45-84aae8a0f303"
-      (reference "#PWR0247") (unit 1) (value "+5V") (footprint "")
-    )
-    (path "/dd09b3c7-f3f1-4702-9c67-cfc029c2d128/30846e71-8b4d-4198-9239-1170998d7a5f"
-      (reference "#PWR0248") (unit 1) (value "GND") (footprint "")
-    )
     (path "/dd09b3c7-f3f1-4702-9c67-cfc029c2d128/75edc28a-fde8-4422-b005-6b6efaaf40ae"
       (reference "#PWR0249") (unit 1) (value "+5V") (footprint "")
@@
       (reference "U203") (unit 1) (value "SN74LXC8T245") (footprint "Package_SO:TSSOP-24_4.4x7.8mm_P0.65mm")
     )
-    (path "/dd09b3c7-f3f1-4702-9c67-cfc029c2d128/c1b5c32d-4c41-4ee7-a564-81f7ea13f012"
-      (reference "U204") (unit 1) (value "SN74LVC2T45") (footprint "Package_SO:VSSOP-8_2.3x2mm_P0.5mm")
-    )
-    (path "/dd09b3c7-f3f1-4702-9c67-cfc029c2d128/16fee360-aff8-446b-9418-9ff8ff763af7"
-      (reference "U205") (unit 1) (value "SN74LVC2T45") (footprint "Package_SO:VSSOP-8_2.3x2mm_P0.5mm")
+    (path "/dd09b3c7-f3f1-4702-9c67-cfc029c2d128/3d5edb30-5108-4cee-bf03-5fbf035fef70"
+      (reference "U206") (unit 1) (value "SN74LXC8T245") (footprint "Package_SO:TSSOP-24_4.4x7.8mm_P0.65mm")
     )
     (path "/d78c8e5b-f415-45d2-97bd-68d83365a2b9/62adabf5-8f35-4e69-8692-db2cbe767550"
