File: blinkenlights/indicators.kicad_sch (KiCad schematic)
At the start: 43 parts, among them U402 74LVC2G34

Commit message: Some more direct IOs for blinkenlights
- /DTACK, /BERR, AS and R/W can be directly read/driven by Teensy GPIO;
  this should allow us to do bus transactions much faster since we can
  prepare the SPI transactions to set up the bus values, then control
  the bus timings most accurately.

- Fixed up a few incorrect pin directions for symbols used in the
  blinkenlights board
Parts:
- U402: footprint Package_TO_SOT_SMD:SOT-23-6_Handsoldering -> Package_TO_SOT_SMD:SOT-363_SC-70-6_Handsoldering
Connections:
- no-connect marks 0 -> 20
Changed lines of the file:
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@@
   (junction (at 72.771 182.9184) (diameter 0) (color 0 0 0 0)
   )
+  (no_connect (at 51.435 169.545))
+  (no_connect (at 152.4 128.905))
+  (no_connect (at 51.435 173.355))
+  (no_connect (at 152.4 169.545))
+  (no_connect (at 99.695 40.005))
+  (no_connect (at 152.4 80.01))
+  (no_connect (at 51.435 80.01))
+  (no_connect (at 51.435 36.195))
+  (no_connect (at 99.695 80.01))
+  (no_connect (at 152.4 173.355))
+  (no_connect (at 51.435 125.095))
+  (no_connect (at 99.695 36.195))
+  (no_connect (at 152.4 40.005))
+  (no_connect (at 99.695 83.82))
+  (no_connect (at 152.4 125.095))
+  (no_connect (at 51.435 40.005))
+  (no_connect (at 51.435 128.905))
+  (no_connect (at 51.435 83.82))
+  (no_connect (at 152.4 36.195))
+  (no_connect (at 152.4 83.82))
   (bus_entry (at 20.32 81.28) (size 2.54 2.54)
     (stroke (width 0) (type default) (color 0 0 0 0))
@@
     (property "Reference" "U402" (id 0) (at 257.175 129.54 0))
     (property "Value" "74LVC2G34" (id 1) (at 257.175 132.08 0))
-    (property "Footprint" "Package_TO_SOT_SMD:SOT-23-6_Handsoldering" (id 2) (at 257.81 137.795 0)
-      (effects (font (size 1.27 1.27)) hide)
-    )
+    (property "Footprint" "Package_TO_SOT_SMD:SOT-363_SC-70-6_Handsoldering" (id 2) (at 257.81 137.795 0)
+      (effects (font (size 1.27 1.27)) hide)
+    )
