File: blinkenlights/io.kicad_sch (KiCad schematic)
At the start: 18 parts, among them U501 XRA1403, U502 PCA9306DP, U503 XRA1403, U504 XRA1402, U505 XRA1403, U506 Teensy4.0

Commit message: Finish routing of blinkenlights board
- Completed routing of the board, including the function code lines and
  other such fun stuff
Parts:
- added C501: 100nF, Capacitor_SMD:C_0805_2012Metric, symbol Device:C_Small
- added U507: 74AUC2G06, Package_TO_SOT_SMD:SOT-23-6_Handsoldering, symbol 74xGxx:74AUC2G06
Connections:
- net +3V3: now also C501.1, U507.5 (VCC), U507.5 (VCC)
- net GND: now also C501.2, U507.2 (GND), U507.2 (GND), U507.3
- net ~{HALT}: now also U507.6
- net ASSERT_HALT: now reaches U506.21 (14_A0_TX3_SPDIF_OUT)
- net ASSERT_HALT: now also U507.1
Changed lines of the file:
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@@
+    (stroke (width 0) (type default) (color 0 0 0 0))
+  )
+  (wire (pts (xy 38.735 140.335) (xy 52.07 140.335))
     (stroke (width 0) (type default) (color 0 0 0 0))
   )
@@
     (stroke (width 0) (type default) (color 0 0 0 0))
   )
+  (wire (pts (xy 66.04 140.335) (xy 79.375 140.335))
+    (stroke (width 0) (type default) (color 0 0 0 0))
+  )
   (wire (pts (xy 210.312 59.69) (xy 203.962 59.69))
     (stroke (width 0) (type default) (color 0 0 0 0))
@@
   )
   (wire (pts (xy 158.75 165.735) (xy 158.75 180.975))
+    (stroke (width 0) (type default) (color 0 0 0 0))
+  )
+  (wire (pts (xy 17.78 80.645) (xy 29.21 80.645))
     (stroke (width 0) (type default) (color 0 0 0 0))
   )
@@
     (effects (font (size 1.27 1.27)) (justify left bottom))
   )
+  (label "~{HALT}" (at 79.375 140.335 180)
+    (effects (font (size 1.27 1.27)) (justify right bottom))
+  )
   (label "D12" (at 203.962 54.61 0)
     (effects (font (size 1.27 1.27)) (justify left bottom))
@@
     (effects (font (size 1.27 1.27)) (justify left bottom))
   )
+  (label "ASSERT_HALT" (at 38.735 140.335 0)
+    (effects (font (size 1.27 1.27)) (justify left bottom))
+  )
   (label "SCK" (at 163.195 91.44 0)
     (effects (font (size 1.27 1.27)) (justify left bottom))
@@
   )
   (label "A22" (at 265.43 91.44 0)
+    (effects (font (size 1.27 1.27)) (justify left bottom))
+  )
+  (label "ASSERT_HALT" (at 17.78 80.645 0)
     (effects (font (size 1.27 1.27)) (justify left bottom))
   )
@@
     )
     (pin "1")
+  )
+  (symbol (lib_id "74xGxx:74AUC2G06") (at 59.69 159.385 0) (unit 2)
+    (in_bom yes) (on_board yes) (fields_autoplaced)
+    (property "Reference" "U507" (id 0) (at 59.055 151.13 0))
+    (property "Value" "74AUC2G06" (id 1) (at 59.055 153.67 0))
+    (property "Footprint" "Package_TO_SOT_SMD:SOT-23-6_Handsoldering" (id 2) (at 59.69 159.385 0)
+      (effects (font (size 1.27 1.27)) hide)
+    )
+    (property "Datasheet" "http://www.ti.com/lit/sg/scyt129e/scyt129e.pdf" (id 3) (at 59.69 159.385 0)
+      (effects (font (size 1.27 1.27)) hide)
+    )
+    (pin "2")
+    (pin "5")
+    (pin "3")
+    (pin "4")
+  )
+  (symbol (lib_id "Device:C_Small") (at 43.815 151.13 0) (unit 1)
+    (in_bom yes) (on_board yes) (fields_autoplaced)
+    (property "Reference" "C501" (id 0) (at 46.1391 150.2215 0)
+      (effects (font (size 1.27 1.27)) (justify left))
+    )
+    (property "Value" "100nF" (id 1) (at 46.1391 152.9966 0)
+      (effects (font (size 1.27 1.27)) (justify left))
+    )
+    (property "Footprint" "Capacitor_SMD:C_0805_2012Metric" (id 2) (at 43.815 151.13 0)
+      (effects (font (size 1.27 1.27)) hide)
+    )
+    (property "Datasheet" "~" (id 3) (at 43.815 151.13 0)
+      (effects (font (size 1.27 1.27)) hide)
+    )
+    (pin "1")
+    (pin "2")
   )
   (symbol (lib_id "power:GND") (at 85.09 90.805 90) (unit 1)
@@
     (pin "9")
   )
+  (symbol (lib_id "power:GND") (at 52.07 159.385 0) (unit 1)
+    (in_bom yes) (on_board yes) (fields_autoplaced)
+    (property "Reference" "#PWR0516" (id 0) (at 52.07 165.735 0)
+      (effects (font (size 1.27 1.27)) hide)
+    )
+    (property "Value" "GND" (id 1) (at 52.07 163.83 0))
+    (property "Footprint" "" (id 2) (at 52.07 159.385 0)
+      (effects (font (size 1.27 1.27)) hide)
+    )
+    (property "Datasheet" "" (id 3) (at 52.07 159.385 0)
+      (effects (font (size 1.27 1.27)) hide)
+    )
+    (pin "1")
+  )
+  (symbol (lib_id "power:GND") (at 59.69 161.925 0) (unit 1)
+    (in_bom yes) (on_board yes) (fields_autoplaced)
+    (property "Reference" "#PWR0520" (id 0) (at 59.69 168.275 0)
+      (effects (font (size 1.27 1.27)) hide)
+    )
+    (property "Value" "GND" (id 1) (at 59.69 166.37 0))
+    (property "Footprint" "" (id 2) (at 59.69 161.925 0)
+      (effects (font (size 1.27 1.27)) hide)
+    )
+    (property "Datasheet" "" (id 3) (at 59.69 161.925 0)
+      (effects (font (size 1.27 1.27)) hide)
+    )
+    (pin "1")
+  )
   (symbol (lib_id "power:GND") (at 173.482 62.23 0) (unit 1)
     (in_bom yes) (on_board yes) (fields_autoplaced)
@@
     (pin "8")
   )
+  (symbol (lib_id "power:GND") (at 59.69 142.875 0) (unit 1)
+    (in_bom yes) (on_board yes) (fields_autoplaced)
+    (property "Reference" "#PWR0518" (id 0) (at 59.69 149.225 0)
+      (effects (font (size 1.27 1.27)) hide)
+    )
+    (property "Value" "GND" (id 1) (at 59.69 147.32 0))
+    (property "Footprint" "" (id 2) (at 59.69 142.875 0)
+      (effects (font (size 1.27 1.27)) hide)
+    )
+    (property "Datasheet" "" (id 3) (at 59.69 142.875 0)
+      (effects (font (size 1.27 1.27)) hide)
+    )
+    (pin "1")
+  )
   (symbol (lib_id "Device:R_Small") (at 164.465 165.735 90) (unit 1)
     (in_bom yes) (on_board yes)
@@
     (pin "2")
   )
+  (symbol (lib_id "power:+3V3") (at 59.69 156.845 270) (unit 1)
+    (in_bom yes) (on_board yes) (fields_autoplaced)
+    (property "Reference" "#PWR0519" (id 0) (at 55.88 156.845 0)
+      (effects (font (size 1.27 1.27)) hide)
+    )
+    (property "Value" "+3V3" (id 1) (at 63.5 156.8449 90)
+      (effects (font (size 1.27 1.27)) (justify left))
+    )
+    (property "Footprint" "" (id 2) (at 59.69 156.845 0)
+      (effects (font (size 1.27 1.27)) hide)
+    )
+    (property "Datasheet" "" (id 3) (at 59.69 156.845 0)
+      (effects (font (size 1.27 1.27)) hide)
+    )
+    (pin "1")
+  )
   (symbol (lib_id "power:GND") (at 29.21 29.845 270) (unit 1)
     (in_bom yes) (on_board yes) (fields_autoplaced)
@@
     (pin "1")
   )
+  (symbol (lib_id "74xGxx:74AUC2G06") (at 59.69 140.335 0) (unit 1)
+    (in_bom yes) (on_board yes) (fields_autoplaced)
+    (property "Reference" "U507" (id 0) (at 59.055 132.08 0))
+    (property "Value" "74AUC2G06" (id 1) (at 59.055 134.62 0))
+    (property "Footprint" "Package_TO_SOT_SMD:SOT-23-6_Handsoldering" (id 2) (at 59.69 140.335 0)
+      (effects (font (size 1.27 1.27)) hide)
+    )
+    (property "Datasheet" "http://www.ti.com/lit/sg/scyt129e/scyt129e.pdf" (id 3) (at 59.69 140.335 0)
+      (effects (font (size 1.27 1.27)) hide)
+    )
+    (pin "2")
+    (pin "5")
+    (pin "1")
+    (pin "6")
+  )
   (symbol (lib_id "power:+3V3") (at 234.95 59.69 90) (unit 1)
     (in_bom yes) (on_board yes) (fields_autoplaced)
@@
     )
     (property "Datasheet" "" (id 3) (at 85.09 47.625 0)
+      (effects (font (size 1.27 1.27)) hide)
+    )
+    (pin "1")
+  )
+  (symbol (lib_id "power:GND") (at 43.815 153.67 0) (unit 1)
+    (in_bom yes) (on_board yes) (fields_autoplaced)
+    (property "Reference" "#PWR0515" (id 0) (at 43.815 160.02 0)
+      (effects (font (size 1.27 1.27)) hide)
+    )
+    (property "Value" "GND" (id 1) (at 43.815 158.115 0))
+    (property "Footprint" "" (id 2) (at 43.815 153.67 0)
+      (effects (font (size 1.27 1.27)) hide)
+    )
+    (property "Datasheet" "" (id 3) (at 43.815 153.67 0)
+      (effects (font (size 1.27 1.27)) hide)
+    )
+    (pin "1")
+  )
+  (symbol (lib_id "power:+3V3") (at 43.815 148.59 0) (unit 1)
+    (in_bom yes) (on_board yes) (fields_autoplaced)
+    (property "Reference" "#PWR0514" (id 0) (at 43.815 152.4 0)
+      (effects (font (size 1.27 1.27)) hide)
+    )
+    (property "Value" "+3V3" (id 1) (at 43.815 142.875 0))
+    (property "Footprint" "" (id 2) (at 43.815 148.59 0)
+      (effects (font (size 1.27 1.27)) hide)
+    )
+    (property "Datasheet" "" (id 3) (at 43.815 148.59 0)
       (effects (font (size 1.27 1.27)) hide)
     )
@@
       (effects (font (size 1.27 1.27)) hide)
     )
+    (pin "1")
+  )
+  (symbol (lib_id "power:+3V3") (at 59.69 137.795 270) (unit 1)
+    (in_bom yes) (on_board yes) (fields_autoplaced)
+    (property "Reference" "#PWR0517" (id 0) (at 55.88 137.795 0)
+      (effects (font (size 1.27 1.27)) hide)
+    )
+    (property "Value" "+3V3" (id 1) (at 63.5 137.7949 90)
+      (effects (font (size 1.27 1.27)) (justify left))
+    )
+    (property "Footprint" "" (id 2) (at 59.69 137.795 0)
+      (effects (font (size 1.27 1.27)) hide)
+    )
+    (property "Datasheet" "" (id 3) (at 59.69 137.795 0)
+      (effects (font (size 1.27 1.27)) hide)
+    )

Commit message: Added a few more test points
- Also, tweaked the package of the I2C translator to be one that's
  actually in stock
Parts:
- added R504: 200k, Resistor_SMD:R_0805_2012Metric, symbol Device:R_Small
- U502: footprint Package_SO:TSSOP-8_3x3mm_P0.65mm -> Package_SO:SO-8_3.9x4.9mm_P1.27mm
- U507: value 74AUC2G06 -> 74LVC2G06
- U507: value 74AUC2G06 -> 74LVC2G06; symbol 74xGxx:74AUC2G06 -> 74xGxx:74LVC2G06; MPN (none) -> SN74LVC2G06DBVR
Connections:
- net +5V: now also R504.2
- net at R501.1, U502.7 (VREF2): no longer U502.8 (EN)
- net ~{I2C_BUF_DIS}: now reaches U505.13 (P8)
- net ~{I2C_BUF_DIS}: now also U502.8 (EN), R504.1

Commit message: Replaced many B case caps with A case
- There were sufficiently many 5V tantalum capcaitors on the
  blinkenlights board with the B case footprint (for 25V) rather than
  the A case (for 16V) assigned.
Parts:
- C514: footprint Capacitor_Tantalum_SMD:CP_EIA-3528-21_Kemet-B -> Capacitor_Tantalum_SMD:CP_EIA-3216-18_Kemet-A
Changed lines of the file:
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@@
       (effects (font (size 1.27 1.27)) (justify left))
     )
-    (property "Footprint" "Capacitor_Tantalum_SMD:CP_EIA-3528-21_Kemet-B" (id 2) (at 273.685 155.575 0)
+    (property "Footprint" "Capacitor_Tantalum_SMD:CP_EIA-3216-18_Kemet-A" (id 2) (at 273.685 155.575 0)
       (effects (font (size 1.27 1.27)) hide)
     )
