File: backplane-breakout/backplane-breakout.kicad_pcb (KiCad board)
At the start: 2 copper layers, 100 x 100 mm, 12 parts, among them J101 Backplane

Commit message: Finished backplane breakout
- All of the backplane signals (for an expansion card) are brought out
  to 2x10 headers, which can connect to the logic analyzer through
  isolation adapters or direct probing in a more compact pinout

- Added a footprint for a shrouded 2x10 header
Parts:
- added J102: Conn_02x10_Odd_Even, 68komputer-common:Shrouded_PinHeader_2x10_P2.54mm_Vertical, B.Cu at (88.9, 92.0)
- added J103: Conn_02x10_Odd_Even, 68komputer-common:Shrouded_PinHeader_2x10_P2.54mm_Vertical, B.Cu at (89.0, 71.6)
- added J104: Conn_02x10_Odd_Even, 68komputer-common:Shrouded_PinHeader_2x10_P2.54mm_Vertical, B.Cu at (89.0, 56.2)
- added J105: Conn_02x10_Odd_Even, 68komputer-common:Shrouded_PinHeader_2x10_P2.54mm_Vertical, B.Cu at (89.0, 40.8)
- added TP101: CLK, TestPoint:TestPoint_Keystone_5000-5004_Miniature, B.Cu at (49.1, 53.2)
- added TP102: GND, TestPoint:TestPoint_Keystone_5000-5004_Miniature, B.Cu at (49.1, 58.4)
- added TP103: +12V, TestPoint:TestPoint_Keystone_5000-5004_Miniature, B.Cu at (42.8, 108.8)
- added TP104: +5V, TestPoint:TestPoint_Keystone_5000-5004_Miniature, B.Cu at (42.8, 116.1)
- added TP105: GND, TestPoint:TestPoint_Keystone_5000-5004_Miniature, B.Cu at (52.7, 108.8)
Connections:
- J101 pad a32: /SNDR -> GND
- J101 pad c32: /SNDL -> GND
Routing:
- net /CLK: track 0.00 -> 127.9 mm, vias 0 -> 1
- net /A10: track 0.00 -> 84.9 mm, vias 0 -> 1
- net /A8: track 0.00 -> 84.4 mm, vias 0 -> 1
- net /A5: track 0.00 -> 84.3 mm, vias 0 -> 1
- net /A7: track 0.00 -> 84.2 mm, vias 0 -> 1
- net /A14: track 0.00 -> 83.7 mm, vias 0 -> 1
- net /A3: track 0.00 -> 83.6 mm, vias 0 -> 1
- net /A1: track 0.00 -> 82.8 mm, vias 0 -> 1
- net /A11: track 0.00 -> 81.1 mm, vias 0 -> 1
- net /~{BG}: track 0.00 -> 80.7 mm, vias 0 -> 1
- net /A12: track 0.00 -> 80.6 mm, vias 0 -> 1
- net /A9: track 0.00 -> 80.5 mm, vias 0 -> 1
- net /A13: track 0.00 -> 80.4 mm, vias 0 -> 1
- net /~{RESET}: track 0.00 -> 80.1 mm, vias 0 -> 1
- net /A6: track 0.00 -> 79.4 mm, vias 0 -> 1
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- added copper zone on F.Cu, net GND
Other:
- board text added: "Address/Bus Ctrl"
- board text added: "Data"
- board text added: "JLCJLCJLCJLC"
- board text added: "Misc"
