File: backplane/Audio.kicad_sch (KiCad schematic)
At the start: 8 parts, among them U701 LM833

Commit message: Minor tweaks to all boards
- Moved around some traces on the 68000 CPU card for prettiness

- Added a connector on the backplane to provide +5V/+12V without a
  management card installed (for testing)
Other:
- company: (none) -> Tristan Seifert
- title: (none) -> Backplane
Changed lines of the file:
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@@
 (kicad_sch (version 20211123) (generator eeschema)
   (paper "A4")
+  (title_block
+    (title "Backplane")
+    (date "2022-01-09")
+    (rev "1")
+    (company "Tristan Seifert")
+  )
   (junction (at 264.795 141.605) (diameter 0) (color 0 0 0 0)
   )
