File: backplane/Management.kicad_sch (KiCad schematic)
At the start: 7 parts, among them J201 Management

Commit message: Minor tweaks to all boards
- Moved around some traces on the 68000 CPU card for prettiness

- Added a connector on the backplane to provide +5V/+12V without a
  management card installed (for testing)
Parts:
- added J202: Screw_Terminal_01x03, Connector_Phoenix_MC:PhoenixContact_MCV_1,5_3-GF-3.5_1x03_P3.50mm_Vertical_ThreadedFlange_MountHole, symbol Connector:Screw_Terminal_01x03
Connections:
- net +12V: now also J202.1 (Pin_1)
- net +5V: now also J202.3 (Pin_3)
- net GND: now also J202.2 (Pin_2)
Other:
- company: (none) -> Tristan Seifert
- title: (none) -> Backplane
Changed lines of the file:
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@@
 (kicad_sch (version 20211123) (generator eeschema)
   (paper "A4")
+  (title_block
+    (title "Backplane")
+    (date "2022-01-09")
+    (rev "1")
+    (company "Tristan Seifert")
+    (comment 1 "J202 is optional; for powering backplane w/o management card")
+  )
   (junction (at 269.875 22.86) (diameter 0) (color 0 0 0 0)
   )
@@
     (pin "1")
   )
+  (symbol (lib_id "power:GND") (at 267.97 154.94 270) (mirror x) (unit 1)
+    (in_bom yes) (on_board yes) (fields_autoplaced)
+    (property "Reference" "#PWR0132" (id 0) (at 261.62 154.94 0)
+      (effects (font (size 1.27 1.27)) hide)
+    )
+    (property "Value" "GND" (id 1) (at 264.795 155.419 90)
+      (effects (font (size 1.27 1.27)) (justify right))
+    )
+    (property "Footprint" "" (id 2) (at 267.97 154.94 0)
+      (effects (font (size 1.27 1.27)) hide)
+    )
+    (property "Datasheet" "" (id 3) (at 267.97 154.94 0)
+      (effects (font (size 1.27 1.27)) hide)
+    )
+    (pin "1")
+  )
   (symbol (lib_id "power:+12V") (at 269.875 33.02 90) (unit 1)
     (in_bom yes) (on_board yes) (fields_autoplaced)
@@
     (pin "1")
   )
+  (symbol (lib_id "power:+12V") (at 267.97 152.4 90) (mirror x) (unit 1)
+    (in_bom yes) (on_board yes) (fields_autoplaced)
+    (property "Reference" "#PWR0133" (id 0) (at 271.78 152.4 0)
+      (effects (font (size 1.27 1.27)) hide)
+    )
+    (property "Value" "+12V" (id 1) (at 264.795 152.879 90)
+      (effects (font (size 1.27 1.27)) (justify left))
+    )
+    (property "Footprint" "" (id 2) (at 267.97 152.4 0)
+      (effects (font (size 1.27 1.27)) hide)
+    )
+    (property "Datasheet" "" (id 3) (at 267.97 152.4 0)
+      (effects (font (size 1.27 1.27)) hide)
+    )
+    (pin "1")
+  )
+  (symbol (lib_id "Connector:Screw_Terminal_01x03") (at 273.05 154.94 0) (unit 1)
+    (in_bom yes) (on_board yes) (fields_autoplaced)
+    (property "Reference" "J202" (id 0) (at 273.05 147.1635 0))
+    (property "Value" "Screw_Terminal_01x03" (id 1) (at 273.05 149.9386 0))
+    (property "Footprint" "Connector_Phoenix_MC:PhoenixContact_MCV_1,5_3-GF-3.5_1x03_P3.50mm_Vertical_ThreadedFlange_MountHole" (id 2) (at 273.05 154.94 0)
+      (effects (font (size 1.27 1.27)) hide)
+    )
+    (property "Datasheet" "~" (id 3) (at 273.05 154.94 0)
+      (effects (font (size 1.27 1.27)) hide)
+    )
+    (property "MPN" "1843237" (id 4) (at 273.05 154.94 0)
+      (effects (font (size 1.27 1.27)) hide)
+    )
+    (pin "1")
+    (pin "2")
+    (pin "3")
+  )
   (symbol (lib_id "power:GND") (at 269.875 35.56 270) (unit 1)
     (in_bom yes) (on_board yes) (fields_autoplaced)
@@
       (effects (font (size 1.27 1.27)) hide)
     )
+    (pin "1")
+  )
+  (symbol (lib_id "power:+5V") (at 267.97 157.48 90) (mirror x) (unit 1)
+    (in_bom yes) (on_board yes) (fields_autoplaced)
+    (property "Reference" "#PWR0131" (id 0) (at 271.78 157.48 0)
+      (effects (font (size 1.27 1.27)) hide)
+    )
+    (property "Value" "+5V" (id 1) (at 264.795 157.959 90)
+      (effects (font (size 1.27 1.27)) (justify left))
+    )
+    (property "Footprint" "" (id 2) (at 267.97 157.48 0)
+      (effects (font (size 1.27 1.27)) hide)
+    )
+    (property "Datasheet" "" (id 3) (at 267.97 157.48 0)
+      (effects (font (size 1.27 1.27)) hide)
+    )

Commit message: Switched remaining pluggable screw terminals
- Replaced the pluggable/replaceable screw terminals with CUI devices
  parts on the backplane (+12V/GND/+5V) and relay board (switched
  contacts) since they're much cheaper and basically the same thing as
  the corresponding WE/Phoenix Contact parts
Parts:
- J202: footprint Connector_Phoenix_MC:PhoenixContact_MCV_1,5_3-GF-3.5_1x03_P3.50mm_Vertical_ThreadedFlange_MountHole -> 68komputer-common:CUI_TBP02R2W-381-03BE; MPN 1843237 -> TBP02R2W-381-03BE; MPN2 (none) -> TBP02P1W-381-03BE
Changed lines of the file:
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@@
     (property "Reference" "J202" (id 0) (at 273.05 147.1635 0))
     (property "Value" "Screw_Terminal_01x03" (id 1) (at 273.05 149.9386 0))
-    (property "Footprint" "Connector_Phoenix_MC:PhoenixContact_MCV_1,5_3-GF-3.5_1x03_P3.50mm_Vertical_ThreadedFlange_MountHole" (id 2) (at 273.05 154.94 0)
+    (property "Footprint" "68komputer-common:CUI_TBP02R2W-381-03BE" (id 2) (at 273.05 154.94 0)
       (effects (font (size 1.27 1.27)) hide)
     )
@@
       (effects (font (size 1.27 1.27)) hide)
     )
-    (property "MPN" "1843237" (id 4) (at 273.05 154.94 0)
+    (property "MPN" "TBP02R2W-381-03BE" (id 4) (at 273.05 154.94 0)
       (effects (font (size 1.27 1.27)) hide)
     )
+    (property "MPN2" "TBP02P1W-381-03BE" (id 5) (at 273.05 154.94 0)
+      (effects (font (size 1.27 1.27)) hide)
+    )
