File: backplane/slots1.kicad_sch (KiCad schematic)
At the start: 22 parts, among them J501 Slot 1, J502 Slot 4, J503 Slot 2, J504 Slot 3

Commit message: More backplane work
- Added pull up/down resistors at end of board to bring the various
  data/address lines to a controlled state, rather than floating, and
  attempt to control reflections

- Added a clock buffer so each slot gets its own nice buffered clock.

  The clock buffer used is only 1:5 fanout, so the last two slots share
  a clock line.
Connections:
- removed net CLK: J501.a24 (Pin_a24), J502.a24 (Pin_a24), J503.a24 (Pin_a24), J504.a24 (Pin_a24)
- new net CLK0: J501.a24 (Pin_a24)
- new net CLK1: J503.a24 (Pin_a24)
- new net CLK2: J504.a24 (Pin_a24)
- new net CLK3: J502.a24 (Pin_a24)
Changed lines of the file:
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@@
-    (stroke (width 0) (type default) (color 0 0 0 0))
-  )
-  (wire (pts (xy 33.655 83.185) (xy 34.925 83.185))
     (stroke (width 0) (type default) (color 0 0 0 0))
   )
@@
     (stroke (width 0) (type default) (color 0 0 0 0))
   )
-  (wire (pts (xy 33.655 174.625) (xy 34.925 174.625))
+  (wire (pts (xy 28.575 174.625) (xy 34.925 174.625))
     (stroke (width 0) (type default) (color 0 0 0 0))
   )
@@
     (stroke (width 0) (type default) (color 0 0 0 0))
   )
-  (wire (pts (xy 215.9 83.185) (xy 217.17 83.185))
-    (stroke (width 0) (type default) (color 0 0 0 0))
-  )
   (bus (pts (xy 74.93 31.115) (xy 74.93 32.385))
     (stroke (width 0) (type default) (color 0 0 0 0))
@@
     (stroke (width 0) (type default) (color 0 0 0 0))
   )
+  (wire (pts (xy 28.575 83.185) (xy 34.925 83.185))
+    (stroke (width 0) (type default) (color 0 0 0 0))
+  )
+  (wire (pts (xy 210.82 83.185) (xy 217.17 83.185))
+    (stroke (width 0) (type default) (color 0 0 0 0))
+  )
   (wire (pts (xy 34.925 32.385) (xy 34.925 34.925))
     (stroke (width 0) (type default) (color 0 0 0 0))
@@
     (stroke (width 0) (type default) (color 0 0 0 0))
   )
-  (wire (pts (xy 114.3 83.185) (xy 115.57 83.185))
+  (wire (pts (xy 109.22 83.185) (xy 115.57 83.185))
     (stroke (width 0) (type default) (color 0 0 0 0))
   )
@@
     (effects (font (size 1.27 1.27)) (justify right bottom))
   )
+  (label "CLK1" (at 109.22 83.185 0)
+    (effects (font (size 1.27 1.27)) (justify left bottom))
+  )
   (label "D0" (at 47.625 50.165 0)
     (effects (font (size 1.27 1.27)) (justify left bottom))
@@
     (effects (font (size 1.27 1.27)) (justify right bottom))
   )
+  (label "CLK2" (at 210.82 83.185 0)
+    (effects (font (size 1.27 1.27)) (justify left bottom))
+  )
   (label "A[1..23]" (at 56.515 167.005 0)
     (effects (font (size 1.27 1.27)) (justify left bottom))
@@
     (effects (font (size 1.27 1.27)) (justify right bottom))
   )
+  (label "CLK0" (at 28.575 83.185 0)
+    (effects (font (size 1.27 1.27)) (justify left bottom))
+  )
   (label "A23" (at 34.925 146.685 180)
     (effects (font (size 1.27 1.27)) (justify right bottom))
@@
     (effects (font (size 1.27 1.27)) (justify left bottom))
   )
-  (hierarchical_label "CLK" (shape output) (at 215.9 83.185 180)
-    (effects (font (size 1.27 1.27)) (justify right))
+  (label "CLK3" (at 28.575 174.625 0)
+    (effects (font (size 1.27 1.27)) (justify left bottom))
   )
   (hierarchical_label "~{BGACK}" (shape output) (at 158.115 95.885 180)
@@
     (effects (font (size 1.27 1.27)) (justify right))
   )
-  (hierarchical_label "CLK" (shape output) (at 33.655 83.185 180)
-    (effects (font (size 1.27 1.27)) (justify right))
-  )
   (hierarchical_label "FC[0..2]" (shape bidirectional) (at 26.035 177.8 180)
     (effects (font (size 1.27 1.27)) (justify right))
@@
     (effects (font (size 1.27 1.27)) (justify right))
   )
+  (hierarchical_label "CLK[0..3]" (shape input) (at 179.07 113.665 0)
+    (effects (font (size 1.27 1.27)) (justify left))
+  )
   (hierarchical_label "~{UDS}" (shape bidirectional) (at 77.47 78.105 180)
     (effects (font (size 1.27 1.27)) (justify right))
@@
     (effects (font (size 1.27 1.27)) (justify right))
   )
-  (hierarchical_label "CLK" (shape output) (at 114.3 83.185 180)
-    (effects (font (size 1.27 1.27)) (justify right))
-  )
   (hierarchical_label "~{AS}" (shape bidirectional) (at 77.47 80.645 180)
     (effects (font (size 1.27 1.27)) (justify right))
@@
     (effects (font (size 1.27 1.27)) (justify right))
   )
-  (hierarchical_label "CLK" (shape output) (at 33.655 174.625 180)
-    (effects (font (size 1.27 1.27)) (justify right))
-  )

Commit message: Added audio mixer to backplane
- Implemented mixing (via resistors and an op amp) for the audio outputs
  from each slot and CPU card. These inputs are tied to ground through
  weak pull downs, so peripherals can leave the pins open if they're not
  being used.

  It's possible that the resistance values for the mixer aren't quite
  correct and will produce a distorted mess with many peripherals
  outputting sound simultaneously; if that's an issue, we can adjust the
  value of the resistors or add per slot trimmers to adjust each slots'
  relative volume.
Connections:
- net SNDL2: now also J504.c32 (Pin_c32); no longer J502.c32 (Pin_c32)
- net SNDL3: now also J502.c32 (Pin_c32); no longer J504.c32 (Pin_c32)
- net SNDR2: now also J504.a32 (Pin_a32); no longer J502.a32 (Pin_a32)
- net SNDR3: now also J502.a32 (Pin_a32); no longer J504.a32 (Pin_a32)
Changed lines of the file:
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@@
     (effects (font (size 1.27 1.27)) (justify left bottom))
   )
-  (label "SNDR3" (at 217.17 103.505 180)
+  (label "SNDR2" (at 217.17 103.505 180)
     (effects (font (size 1.27 1.27)) (justify right bottom))
   )
@@
     (effects (font (size 1.27 1.27)) (justify right bottom))
   )
-  (label "SNDL2" (at 83.82 194.945 180)
+  (label "SNDL3" (at 83.82 194.945 180)
     (effects (font (size 1.27 1.27)) (justify right bottom))
   )
@@
     (effects (font (size 1.27 1.27)) (justify right bottom))
   )
-  (label "SNDL3" (at 266.065 103.505 180)
+  (label "SNDL2" (at 266.065 103.505 180)
     (effects (font (size 1.27 1.27)) (justify right bottom))
   )
@@
     (effects (font (size 1.27 1.27)) (justify right bottom))
   )
-  (label "SNDR2" (at 34.925 194.945 180)
+  (label "SNDR3" (at 34.925 194.945 180)
     (effects (font (size 1.27 1.27)) (justify right bottom))
   )

Commit message: Backplane mechanical improvements
- Added screw holes to the backplane; they may or may not actually be
  correct but the spacing between them should be right. We've got holes
  every two HU's (2x .2") for extra spacing/material between holes

- Added reset LED and some more pull ups

- Minor tweaks to backplane management card
Parts:
- added R501: 0R, Resistor_SMD:R_0805_2012Metric, symbol Device:R_Small
Connections:
- net GND: now also R501.1
- net ~{IRQ_IN_1}: now also R501.2
Changed lines of the file:
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@@
     (stroke (width 0) (type default) (color 0 0 0 0))
   )
+  (wire (pts (xy 129.54 120.65) (xy 116.84 120.65))
+    (stroke (width 0) (type default) (color 0 0 0 0))
+  )
   (bus (pts (xy 208.28 52.705) (xy 208.28 57.785))
     (stroke (width 0) (type default) (color 0 0 0 0))
@@
     (effects (font (size 1.27 1.27)) (justify right bottom))
   )
+  (label "~{IRQ_IN_1}" (at 129.54 120.65 180)
+    (effects (font (size 1.27 1.27)) (justify right bottom))
+  )
   (label "D8" (at 229.87 34.925 0)
     (effects (font (size 1.27 1.27)) (justify left bottom))
@@
     (pin "1")
   )
+  (symbol (lib_id "Device:R_Small") (at 114.3 120.65 90) (unit 1)
+    (in_bom yes) (on_board yes) (fields_autoplaced)
+    (property "Reference" "R501" (id 0) (at 114.3 114.935 90))
+    (property "Value" "0R" (id 1) (at 114.3 117.475 90))
+    (property "Footprint" "Resistor_SMD:R_0805_2012Metric" (id 2) (at 114.3 120.65 0)
+      (effects (font (size 1.27 1.27)) hide)
+    )
+    (property "Datasheet" "~" (id 3) (at 114.3 120.65 0)
+      (effects (font (size 1.27 1.27)) hide)
+    )
+    (property "MPN" "RC0805JR-100RL" (id 4) (at 114.3 120.65 90)
+      (effects (font (size 1.27 1.27)) hide)
+    )
+    (pin "1")
+    (pin "2")
+  )
   (symbol (lib_id "68komputer-common:Conn_03x32_Row_Letter_First") (at 172.085 62.865 0) (mirror y) (unit 2)
     (in_bom yes) (on_board yes)
@@
       (effects (font (size 1.27 1.27)) hide)
     )
+    (pin "1")
+  )
+  (symbol (lib_id "power:GND") (at 111.76 120.65 0) (unit 1)
+    (in_bom yes) (on_board yes) (fields_autoplaced)
+    (property "Reference" "#PWR0597" (id 0) (at 111.76 127 0)
+      (effects (font (size 1.27 1.27)) hide)
+    )
+    (property "Value" "GND" (id 1) (at 111.76 125.2125 0))
+    (property "Footprint" "" (id 2) (at 111.76 120.65 0)
+      (effects (font (size 1.27 1.27)) hide)
+    )
+    (property "Datasheet" "" (id 3) (at 111.76 120.65 0)
+      (effects (font (size 1.27 1.27)) hide)
+    )

Commit message: Minor tweaks to all boards
- Moved around some traces on the 68000 CPU card for prettiness

- Added a connector on the backplane to provide +5V/+12V without a
  management card installed (for testing)
Other:
- company: (none) -> Tristan Seifert
- title: (none) -> Backplane
Changed lines of the file:
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@@
 (kicad_sch (version 20211123) (generator eeschema)
   (paper "A4")
+  (title_block
+    (title "Backplane")
+    (date "2022-01-09")
+    (rev "1")
+    (company "Tristan Seifert")
+  )
   (junction (at 181.61 137.16) (diameter 0) (color 0 0 0 0)
   )
