File: backplane_mgmt/vreg-12v.kicad_sch (KiCad schematic)
At the start: 26 parts, among them Q401 PSMN045-80YS, Q402 PSMN045-80YS, U401 LM25116

Commit message: Minor layout tweaks across the board
- Added an input for a test clock, and a jumper for sending this clock
  instead of the CPU clock to the clock pins of the expansion cards on
  the backplane boards

- Reworked a bunch of the power supply board

- Minor changes (to consolidate BOMs) on CPU board for some capacitors,
  they were replaced with SMD versions
Other:
- moved on the sheet: C401, C402, C403, C404, C405, C406, C407, C408, C409, C410, C411, C412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
